File: hardware/bridge/kicad/01b_usb_limit.kicad_sch (KiCad schematic)
At the start: 5 parts, among them U3 TPS2553QDBVRQ1

Commit message: fix: close hardware rail-fault paths and sensor contract gaps
Parts:
- removed C4: 1u, CANView:Capacitor_SMD__C_0603_1608Metric, symbol CANView:CANView_bridge_C4
- removed C5: 1u, CANView:Capacitor_SMD__C_0603_1608Metric, symbol CANView:CANView_bridge_C5
- removed R4: 26.7k, CANView:Resistor_SMD__R_0402_1005Metric, symbol CANView:CANView_bridge_R4
- added C6: 1u, CANView:Capacitor_SMD__C_0603_1608Metric, symbol CANView:CANView_bridge_C6
- added C7: 1u, CANView:Capacitor_SMD__C_0603_1608Metric, symbol CANView:CANView_bridge_C7
- added R6: 10k, CANView:Resistor_SMD__R_0402_1005Metric, symbol CANView:CANView_bridge_R6
- R5: value 10k -> 26.7k; MPN GEN-R-0402-10k-1% -> GEN-R-0402-26.7k-1%
Connections:
- net GND: now also R5.2, C6.2, C7.2
- net USB_FAULT_N: now also R6.2; no longer R5.2
- net USB_ILIM: now also R5.1
- net USB_LIMITED: now also C7.1
- net USB_VBUS: now also C6.1, R6.1; no longer R5.1
Other:
- moved on the sheet: R5
