File: hardware/bridge/kicad/02_system_power.kicad_sch (KiCad schematic)
At the start: 7 parts, among them U5 TPS629210DRLR

Commit message: fix: close hardware rail-fault paths and sensor contract gaps
Parts:
- removed C6: 4.7u, CANView:Capacitor_SMD__C_0603_1608Metric, symbol CANView:CANView_bridge_C6
- removed C7: 22u, CANView:Capacitor_SMD__C_0805_2012Metric, symbol CANView:CANView_bridge_C7
- removed R6: 0, CANView:Resistor_SMD__R_0805_2012Metric, symbol CANView:CANView_bridge_R6
- added C8: 4.7u, CANView:Capacitor_SMD__C_0603_1608Metric, symbol CANView:CANView_bridge_C8
- added C9: 22u, CANView:Capacitor_SMD__C_0805_2012Metric, symbol CANView:CANView_bridge_C9
- added R9: 27.4k, CANView:Resistor_SMD__R_0402_1005Metric, symbol CANView:CANView_bridge_R9
- R7: value 249k -> 0; footprint CANView:Resistor_SMD__R_0402_1005Metric -> CANView:Resistor_SMD__R_0805_2012Metric; MPN GEN-R-0402-249k-1% -> GEN-R-0805-0-1%; Specification 0.1W; 50V; ±1%; ±100ppm/K; -55..155C -> 0.25W; 50V; ±1%; ±100ppm/K; -55..155C
- R8: value 27.4k -> 249k; MPN GEN-R-0402-27.4k-1% -> GEN-R-0402-249k-1%
Connections:
- net 3V3: now also C9.1
- net GND: now also C8.2, C9.2, R9.2; no longer R7.2
- net SYS5V: now also R7.2, C8.1
- net SYS_MODE: now also R9.1; no longer R8.1
- net USB_LIMITED: now also R7.1
- net VSET_3V3: now also R8.1; no longer R7.1
Other:
- moved on the sheet: R7, R8
