File: hardware/bridge/kicad/03_reset.kicad_sch (KiCad schematic)
At the start: 4 parts, among them SW1 RESET, U6 TLV803EA30DPWR

Commit message: fix: close hardware rail-fault paths and sensor contract gaps
Parts:
- removed C8: 100n, CANView:Capacitor_SMD__C_0402_1005Metric, symbol CANView:CANView_bridge_C8
- removed R9: 10k, CANView:Resistor_SMD__R_0402_1005Metric, symbol CANView:CANView_bridge_R9
- added C10: 100n, CANView:Capacitor_SMD__C_0402_1005Metric, symbol CANView:CANView_bridge_C10
- added R10: 10k, CANView:Resistor_SMD__R_0402_1005Metric, symbol CANView:CANView_bridge_R10
Connections:
- net 3V3: now also C10.1, R10.1
- net GND: now also C10.2
- net SYS_RESET_N: now also R10.2
Changed lines of the file:
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@@
 (wire (pts (xy 114.3000 55.8800) (xy 121.9200 55.8800)) (stroke (width 0) (type default)))
 (global_label "3V3" (shape bidirectional) (at 121.9200 55.8800 0) (effects (font (size 0.95 0.95)) (justify left)) (property "Intersheetrefs" "${INTERSHEET_REFS}" (at 121.9200 55.8800 0) (hide yes) (effects (font (size 1.0 1.0)) )))
-(symbol (lib_id "CANView:CANView_bridge_R9") (at 50.8000 96.5200 0) (unit 1) (in_bom yes) (on_board yes) (dnp no) (property "Reference" "R9" (at 50.8000 88.9000 0)  (effects (font (size 1.0 1.0)) ))(property "Value" "10k" (at 50.8000 91.4400 0)  (effects (font (size 1.0 1.0)) ))(property "Footprint" "CANView:Resistor_SMD__R_0402_1005Metric" (at 50.8000 96.5200 0) (hide yes) (effects (font (size 1.0 1.0)) ))(property "MPN" "GEN-R-0402-10k-1%" (at 50.8000 96.5200 0) (hide yes) (effects (font (size 1.0 1.0)) ))(property "Specification" "0.1W; 50V; ±1%; ±100ppm/K; -55..155C" (at 50.8000 96.5200 0) (hide yes) (effects (font (size 1.0 1.0)) ))(property "Source" "" (at 50.8000 96.5200 0) (hide yes) (effects (font (size 1.0 1.0)) ))(property "Assembly" "FIT" (at 50.8000 96.5200 0) (hide yes) (effects (font (size 1.0 1.0)) ))(instances (project "bridge" (path "/695535dc-1835-5369-a035-dbad415d33c6/7ded663d-8fba-56a2-80cd-53907fe8a829" (reference "R9") (unit 1)))))
+(symbol (lib_id "CANView:CANView_bridge_R10") (at 50.8000 96.5200 0) (unit 1) (in_bom yes) (on_board yes) (dnp no) (property "Reference" "R10" (at 50.8000 88.9000 0)  (effects (font (size 1.0 1.0)) ))(property "Value" "10k" (at 50.8000 91.4400 0)  (effects (font (size 1.0 1.0)) ))(property "Footprint" "CANView:Resistor_SMD__R_0402_1005Metric" (at 50.8000 96.5200 0) (hide yes) (effects (font (size 1.0 1.0)) ))(property "MPN" "GEN-R-0402-10k-1%" (at 50.8000 96.5200 0) (hide yes) (effects (font (size 1.0 1.0)) ))(property "Specification" "0.1W; 50V; ±1%; ±100ppm/K; -55..155C" (at 50.8000 96.5200 0) (hide yes) (effects (font (size 1.0 1.0)) ))(property "Source" "" (at 50.8000 96.5200 0) (hide yes) (effects (font (size 1.0 1.0)) ))(property "Assembly" "FIT" (at 50.8000 96.5200 0) (hide yes) (effects (font (size 1.0 1.0)) ))(instances (project "bridge" (path "/695535dc-1835-5369-a035-dbad415d33c6/7ded663d-8fba-56a2-80cd-53907fe8a829" (reference "R10") (unit 1)))))
 (wire (pts (xy 40.6400 96.5200) (xy 33.0200 96.5200)) (stroke (width 0) (type default)))
 (global_label "3V3" (shape bidirectional) (at 33.0200 96.5200 180) (effects (font (size 0.95 0.95)) (justify right)) (property "Intersheetrefs" "${INTERSHEET_REFS}" (at 33.0200 96.5200 0) (hide yes) (effects (font (size 1.0 1.0)) )))
 (wire (pts (xy 60.9600 96.5200) (xy 68.5800 96.5200)) (stroke (width 0) (type default)))
 (global_label "SYS_RESET_N" (shape bidirectional) (at 68.5800 96.5200 0) (effects (font (size 0.95 0.95)) (justify left)) (property "Intersheetrefs" "${INTERSHEET_REFS}" (at 68.5800 96.5200 0) (hide yes) (effects (font (size 1.0 1.0)) )))
-(symbol (lib_id "CANView:CANView_bridge_C8") (at 142.2400 96.5200 0) (unit 1) (in_bom yes) (on_board yes) (dnp no) (property "Reference" "C8" (at 142.2400 88.9000 0)  (effects (font (size 1.0 1.0)) ))(property "Value" "100n" (at 142.2400 91.4400 0)  (effects (font (size 1.0 1.0)) ))(property "Footprint" "CANView:Capacitor_SMD__C_0402_1005Metric" (at 142.2400 96.5200 0) (hide yes) (effects (font (size 1.0 1.0)) ))(property "MPN" "GEN-C-0402-100n-16V-X7R" (at 142.2400 96.5200 0) (hide yes) (effects (font (size 1.0 1.0)) ))(property "Specification" "16V; ±10%; X7R; -55..125C; verify effective capacitance under DC bias" (at 142.2400 96.5200 0) (hide yes) (effects (font (size 1.0 1.0)) ))(property "Source" "" (at 142.2400 96.5200 0) (hide yes) (effects (font (size 1.0 1.0)) ))(property "Assembly" "FIT" (at 142.2400 96.5200 0) (hide yes) (effects (font (size 1.0 1.0)) ))(instances (project "bridge" (path "/695535dc-1835-5369-a035-dbad415d33c6/7ded663d-8fba-56a2-80cd-53907fe8a829" (reference "C8") (unit 1)))))
+(symbol (lib_id "CANView:CANView_bridge_C10") (at 142.2400 96.5200 0) (unit 1) (in_bom yes) (on_board yes) (dnp no) (property "Reference" "C10" (at 142.2400 88.9000 0)  (effects (font (size 1.0 1.0)) ))(property "Value" "100n" (at 142.2400 91.4400 0)  (effects (font (size 1.0 1.0)) ))(property "Footprint" "CANView:Capacitor_SMD__C_0402_1005Metric" (at 142.2400 96.5200 0) (hide yes) (effects (font (size 1.0 1.0)) ))(property "MPN" "GEN-C-0402-100n-16V-X7R" (at 142.2400 96.5200 0) (hide yes) (effects (font (size 1.0 1.0)) ))(property "Specification" "16V; ±10%; X7R; -55..125C; verify effective capacitance under DC bias" (at 142.2400 96.5200 0) (hide yes) (effects (font (size 1.0 1.0)) ))(property "Source" "" (at 142.2400 96.5200 0) (hide yes) (effects (font (size 1.0 1.0)) ))(property "Assembly" "FIT" (at 142.2400 96.5200 0) (hide yes) (effects (font (size 1.0 1.0)) ))(instances (project "bridge" (path "/695535dc-1835-5369-a035-dbad415d33c6/7ded663d-8fba-56a2-80cd-53907fe8a829" (reference "C10") (unit 1)))))
 (wire (pts (xy 132.0800 96.5200) (xy 124.4600 96.5200)) (stroke (width 0) (type default)))
 (global_label "3V3" (shape bidirectional) (at 124.4600 96.5200 180) (effects (font (size 0.95 0.95)) (justify right)) (property "Intersheetrefs" "${INTERSHEET_REFS}" (at 124.4600 96.5200 0) (hide yes) (effects (font (size 1.0 1.0)) )))

Commit message: Design independent OTA recovery and update N16R8 hardware
Parts:
- SW1: Specification Momentary normally-open; shared MCU reset -> Momentary normally-open; Communicator drives both superviso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
Changed lines of the file:
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@@
 (wire (pts (xy 152.4000 96.5200) (xy 160.0200 96.5200)) (stroke (width 0) (type default)))
 (global_label "GND" (shape bidirectional) (at 160.0200 96.5200 0) (effects (font (size 0.95 0.95)) (justify left)) (property "Intersheetrefs" "${INTERSHEET_REFS}" (at 160.0200 96.5200 0) (hide yes) (effects (font (size 1.0 1.0)) )))
-(symbol (lib_id "CANView:CANView_bridge_SW1") (at 233.6800 96.5200 0) (unit 1) (in_bom yes) (on_board yes) (dnp no) (property "Reference" "SW1" (at 233.6800 88.9000 0)  (effects (font (size 1.0 1.0)) ))(property "Value" "RESET" (at 233.6800 91.4400 0)  (effects (font (size 1.0 1.0)) ))(property "Footprint" "CANView:Button_Switch_SMD__SW_SPST_TL3342" (at 233.6800 96.5200 0) (hide yes) (effects (font (size 1.0 1.0)) ))(property "MPN" "TL3342F160QG" (at 233.6800 96.5200 0) (hide yes) (effects (font (size 1.0 1.0)) ))(property "Specification" "Momentary normally-open; shared MCU reset" (at 233.6800 96.5200 0) (hide yes) (effects (font (size 1.0 1.0)) ))(property "Source" "" (at 233.6800 96.5200 0) (hide yes) (effects (font (size 1.0 1.0)) ))(property "Assembly" "FIT" (at 233.6800 96.5200 0) (hide yes) (effects (font (size 1.0 1.0)) ))(instances (project "bridge" (path "/695535dc-1835-5369-a035-dbad415d33c6/7ded663d-8fba-56a2-80cd-53907fe8a829" (reference "SW1") (unit 1)))))
+(symbol (lib_id "CANView:CANView_bridge_SW1") (at 233.6800 96.5200 0) (unit 1) (in_bom yes) (on_board yes) (dnp no) (property "Reference" "SW1" (at 233.6800 88.9000 0)  (effects (font (size 1.0 1.0)) ))(property "Value" "RESET" (at 233.6800 91.4400 0)  (effects (font (size 1.0 1.0)) ))(property "Footprint" "CANView:Button_Switch_SMD__SW_SPST_TL3342" (at 233.6800 96.5200 0) (hide yes) (effects (font (size 1.0 1.0)) ))(property "MPN" "TL3342F160QG" (at 233.6800 96.5200 0) (hide yes) (effects (font (size 1.0 1.0)) ))(property "Specification" "Momentary normally-open; Communicator drives both supervisor MR inputs, never joins reset outputs" (at 233.6800 96.5200 0) (hide yes) (effects (font (size 1.0 1.0)) ))(property "Source" "" (at 233.6800 96.5200 0) (hide yes) (effects (font (size 1.0 1.0)) ))(property "Assembly" "FIT" (at 233.6800 96.5200 0) (hide yes) (effects (font (size 1.0 1.0)) ))(instances (project "bridge" (path "/695535dc-1835-5369-a035-dbad415d33c6/7ded663d-8fba-56a2-80cd-53907fe8a829" (reference "SW1") (unit 1)))))
 (wire (pts (xy 223.5200 96.5200) (xy 215.9000 96.5200)) (stroke (width 0) (type default)))
 (global_label "SYS_RESET_N" (shape bidirectional) (at 215.9000 96.5200 180) (effects (font (size 0.95 0.95)) (justify right)) (property "Intersheetrefs" "${INTERSHEET_REFS}" (at 215.9000 96.5200 0) (hide yes) (effects (font (size 1.0 1.0)) )))
