File: hardware/communicator/kicad/00b_reverse_ov.kicad_sch (KiCad schematic)
At the start: 11 parts, among them Q1 BUK9Y12-100E, Q2 BUK9Y12-100E, U7 LM74800QDRRRQ1

Commit message: fix: close hardware rail-fault paths and sensor contract gaps
Parts:
- Q1, Q2: value BUK9Y12-100E -> BUK7Y12-100E; MPN BUK9Y12-100E -> BUK7Y12-100E; Source buk9y12-100e: pinout, SOA; lm7480 pp29-32 -> buk7y12-100e:pp1-2,4,10 pinout, DC VGS and SOA; lm7480 pp6,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; Specification 100V N-MOS; LFPAK56; common-source pair; pulse SOA qualific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 -> 100V N-MOS; DC VGS +/-20V; RDSon<=12mohm@10V/25C; LFPAK56; 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
Changed lines of the file:
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@@
 (kicad_sch (version 20250114) (generator "eeschema") (generator_version "10.0") (paper "A3") (title_block (title "CANView / 00b_reverse_ov") (date "2026-09-05") (rev "R1 REVIEW") (company "digitie/canview") (comment 1 "SCHEMATIC REVIEW ONLY - PCB/HIL release gates remain open"))
 (text "LM74800 common-source: HGATE drives INPUT FET; DGATE drives OUTPUT FET; A/OUT both=CS. Exposed pad FLOATS." (at 15.24 15.24 0) (effects (font (size 1.2 1.2)) (justify left)))
-(symbol (lib_id "CANView:CANView_communicator_Q1") (at 254.0000 55.8800 0) (unit 1) (in_bom yes) (on_board yes) (dnp no) (property "Reference" "Q1" (at 254.0000 40.6400 0)  (effects (font (size 1.0 1.0)) ))(property "Value" "BUK9Y12-100E" (at 254.0000 43.1800 0)  (effects (font (size 1.0 1.0)) ))(property "Footprint" "CANView:Package_TO_SOT_SMD__LFPAK56" (at 254.0000 55.8800 0) (hide yes) (effects (font (size 1.0 1.0)) ))(property "MPN" "BUK9Y12-100E" (at 254.0000 55.8800 0) (hide yes) (effects (font (size 1.0 1.0)) ))(property "Specification" "100V N-MOS; LFPAK56; common-source pair; pulse SOA qualification required" (at 254.0000 55.8800 0) (hide yes) (effects (font (size 1.0 1.0)) ))(property "Source" "buk9y12-100e: pinout, SOA; lm7480 pp29-32" (at 254.0000 55.8800 0) (hide yes) (effects (font (size 1.0 1.0)) ))(property "Assembly" "FIT" (at 254.0000 55.8800 0) (hide yes) (effects (font (size 1.0 1.0)) ))(instances (project "communicator" (path "/c8ff26d1-0b80-520e-ae3f-45aa29bfe092/33f8f21b-ef50-563a-949c-b1cbacf0523a" (reference "Q1") (unit 1)))))
+(symbol (lib_id "CANView:CANView_communicator_Q1") (at 254.0000 55.8800 0) (unit 1) (in_bom yes) (on_board yes) (dnp no) (property "Reference" "Q1" (at 254.0000 40.6400 0)  (effects (font (size 1.0 1.0)) ))(property "Value" "BUK7Y12-100E" (at 254.0000 43.1800 0)  (effects (font (size 1.0 1.0)) ))(property "Footprint" "CANView:Package_TO_SOT_SMD__LFPAK56" (at 254.0000 55.8800 0) (hide yes) (effects (font (size 1.0 1.0)) ))(property "MPN" "BUK7Y12-100E" (at 254.0000 55.8800 0) (hide yes) (effects (font (size 1.0 1.0)) ))(property "Specification" "100V N-MOS; DC VGS +/-20V; RDSon<=12mohm@10V/25C; LFPAK56; common-source pair; pulse SOA qualification required" (at 254.0000 55.8800 0) (hide yes) (effects (font (size 1.0 1.0)) ))(property "Source" "buk7y12-100e:pp1-2,4,10 pinout, DC VGS and SOA; lm7480 pp6,29-32" (at 254.0000 55.8800 0) (hide yes) (effects (font (size 1.0 1.0)) ))(property "Assembly" "FIT" (at 254.0000 55.8800 0) (hide yes) (effects (font (size 1.0 1.0)) ))(instances (project "communicator" (path "/c8ff26d1-0b80-520e-ae3f-45aa29bfe092/33f8f21b-ef50-563a-949c-b1cbacf0523a" (reference "Q1") (unit 1)))))
 (wire (pts (xy 228.6000 50.8000) (xy 220.9800 50.8000)) (stroke (width 0) (type default)))
 (global_label "CS" (shape bidirectional) (at 220.9800 50.8000 180) (effects (font (size 0.95 0.95)) (justify right)) (property "Intersheetrefs" "${INTERSHEET_REFS}" (at 220.9800 50.8000 0) (hide yes) (effects (font (size 1.0 1.0)) )))
@@
 (wire (pts (xy 279.4000 55.8800) (xy 287.0200 55.8800)) (stroke (width 0) (type default)))
 (global_label "VBAT_FUSED" (shape bidirectional) (at 287.0200 55.8800 0) (effects (font (size 0.95 0.95)) (justify left)) (property "Intersheetrefs" "${INTERSHEET_REFS}" (at 287.0200 55.8800 0) (hide yes) (effects (font (size 1.0 1.0)) )))
-(symbol (lib_id "CANView:CANView_communicator_Q2") (at 254.0000 111.7600 0) (unit 1) (in_bom yes) (on_board yes) (dnp no) (property "Reference" "Q2" (at 254.0000 96.5200 0)  (effects (font (size 1.0 1.0)) ))(property "Value" "BUK9Y12-100E" (at 254.0000 99.0600 0)  (effects (font (size 1.0 1.0)) ))(property "Footprint" "CANView:Package_TO_SOT_SMD__LFPAK56" (at 254.0000 111.7600 0) (hide yes) (effects (font (size 1.0 1.0)) ))(property "MPN" "BUK9Y12-100E" (at 254.0000 111.7600 0) (hide yes) (effects (font (size 1.0 1.0)) ))(property "Specification" "100V N-MOS; LFPAK56; common-source pair; pulse SOA qualification required" (at 254.0000 111.7600 0) (hide yes) (effects (font (size 1.0 1.0)) ))(property "Source" "buk9y12-100e: pinout, SOA; lm7480 pp29-32" (at 254.0000 111.7600 0) (hide yes) (effects (font (size 1.0 1.0)) ))(property "Assembly" "FIT" (at 254.0000 111.7600 0) (hide yes) (effects (font (size 1.0 1.0)) ))(instances (project "communicator" (path "/c8ff26d1-0b80-520e-ae3f-45aa29bfe092/33f8f21b-ef50-563a-949c-b1cbacf0523a" (reference "Q2") (unit 1)))))
+(symbol (lib_id "CANView:CANView_communicator_Q2") (at 254.0000 111.7600 0) (unit 1) (in_bom yes) (on_board yes) (dnp no) (property "Reference" "Q2" (at 254.0000 96.5200 0)  (effects (font (size 1.0 1.0)) ))(property "Value" "BUK7Y12-100E" (at 254.0000 99.0600 0)  (effects (font (size 1.0 1.0)) ))(property "Footprint" "CANView:Package_TO_SOT_SMD__LFPAK56" (at 254.0000 111.7600 0) (hide yes) (effects (font (size 1.0 1.0)) ))(property "MPN" "BUK7Y12-100E" (at 254.0000 111.7600 0) (hide yes) (effects (font (size 1.0 1.0)) ))(property "Specification" "100V N-MOS; DC VGS +/-20V; RDSon<=12mohm@10V/25C; LFPAK56; common-source pair; pulse SOA qualification required" (at 254.0000 111.7600 0) (hide yes) (effects (font (size 1.0 1.0)) ))(property "Source" "buk7y12-100e:pp1-2,4,10 pinout, DC VGS and SOA; lm7480 pp6,29-32" (at 254.0000 111.7600 0) (hide yes) (effects (font (size 1.0 1.0)) ))(property "Assembly" "FIT" (at 254.0000 111.7600 0) (hide yes) (effects (font (size 1.0 1.0)) ))(instances (project "communicator" (path "/c8ff26d1-0b80-520e-ae3f-45aa29bfe092/33f8f21b-ef50-563a-949c-b1cbacf0523a" (reference "Q2") (unit 1)))))
 (wire (pts (xy 228.6000 106.6800) (xy 220.9800 106.6800)) (stroke (width 0) (type default)))
 (global_label "CS" (shape bidirectional) (at 220.9800 106.6800 180) (effects (font (size 0.95 0.95)) (justify right)) (property "Intersheetrefs" "${INTERSHEET_REFS}" (at 220.9800 106.6800 0) (hide yes) (effects (font (size 1.0 1.0)) )))
