File: hardware/communicator/kicad/01_usb_c.kicad_sch (KiCad schematic)
At the start: 11 parts, among them J1 USB4105-GF-A, U1 TUSB320LAIRWBR, U2 SN74LVC1G04DBVR

Commit message: fix: close hardware rail-fault paths and sensor contract gaps
Connections:
- net USB_VBUS: no longer C15.1, C16.1, R11.1, U1.12 (VDD), U2.5 (VCC)
- new net USB_CC3V3: C15.1, C16.1, R11.1, U1.12 (VDD), U2.5 (VCC)
Changed lines of the file:
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@@
 (global_label "GND" (shape bidirectional) (at 287.0200 71.1200 0) (effects (font (size 0.95 0.95)) (justify left)) (property "Intersheetrefs" "${INTERSHEET_REFS}" (at 287.0200 71.1200 0) (hide yes) (effects (font (size 1.0 1.0)) )))
 (wire (pts (xy 279.4000 76.2000) (xy 287.0200 76.2000)) (stroke (width 0) (type default)))
-(global_label "USB_VBUS" (shape bidirectional) (at 287.0200 76.2000 0) (effects (font (size 0.95 0.95)) (justify left)) (property "Intersheetrefs" "${INTERSHEET_REFS}" (at 287.0200 76.2000 0) (hide yes) (effects (font (size 1.0 1.0)) )))
+(global_label "USB_CC3V3" (shape bidirectional) (at 287.0200 76.2000 0) (effects (font (size 0.95 0.95)) (justify left)) (property "Intersheetrefs" "${INTERSHEET_REFS}" (at 287.0200 76.2000 0) (hide yes) (effects (font (size 1.0 1.0)) )))
 (symbol (lib_id "CANView:CANView_communicator_R10") (at 142.2400 218.4400 0) (unit 1) (in_bom yes) (on_board yes) (dnp no) (property "Reference" "R10" (at 142.2400 210.8200 0)  (effects (font (size 1.0 1.0)) ))(property "Value" "900k" (at 142.2400 213.3600 0)  (effects (font (size 1.0 1.0)) ))(property "Footprint" "CANView:Resistor_SMD__R_0402_1005Metric" (at 142.2400 218.4400 0) (hide yes) (effects (font (size 1.0 1.0)) ))(property "MPN" "GEN-R-0402-900k-1%" (at 142.2400 218.4400 0) (hide yes) (effects (font (size 1.0 1.0)) ))(property "Specification" "0.1W; 50V; ±1%; ±100ppm/K; -55..155C" (at 142.2400 218.4400 0) (hide yes) (effects (font (size 1.0 1.0)) ))(property "Source" "" (at 142.2400 218.4400 0) (hide yes) (effects (font (size 1.0 1.0)) ))(property "Assembly" "FIT" (at 142.2400 218.4400 0) (hide yes) (effects (font (size 1.0 1.0)) ))(instances (project "communicator" (path "/c8ff26d1-0b80-520e-ae3f-45aa29bfe092/7c624ae8-5f0b-5909-af7f-eefe17ebe63c" (reference "R10") (unit 1)))))
 (wire (pts (xy 132.0800 218.4400) (xy 124.4600 218.4400)) (stroke (width 0) (type default)))
@@
 (symbol (lib_id "CANView:CANView_communicator_R11") (at 233.6800 218.4400 0) (unit 1) (in_bom yes) (on_board yes) (dnp no) (property "Reference" "R11" (at 233.6800 210.8200 0)  (effects (font (size 1.0 1.0)) ))(property "Value" "10k" (at 233.6800 213.3600 0)  (effects (font (size 1.0 1.0)) ))(property "Footprint" "CANView:Resistor_SMD__R_0402_1005Metric" (at 233.6800 218.4400 0) (hide yes) (effects (font (size 1.0 1.0)) ))(property "MPN" "GEN-R-0402-10k-1%" (at 233.6800 218.4400 0) (hide yes) (effects (font (size 1.0 1.0)) ))(property "Specification" "0.1W; 50V; ±1%; ±100ppm/K; -55..155C" (at 233.6800 218.4400 0) (hide yes) (effects (font (size 1.0 1.0)) ))(property "Source" "" (at 233.6800 218.4400 0) (hide yes) (effects (font (size 1.0 1.0)) ))(property "Assembly" "FIT" (at 233.6800 218.4400 0) (hide yes) (effects (font (size 1.0 1.0)) ))(instances (project "communicator" (path "/c8ff26d1-0b80-520e-ae3f-45aa29bfe092/7c624ae8-5f0b-5909-af7f-eefe17ebe63c" (reference "R11") (unit 1)))))
 (wire (pts (xy 223.5200 218.4400) (xy 215.9000 218.4400)) (stroke (width 0) (type default)))
-(global_label "USB_VBUS" (shape bidirectional) (at 215.9000 218.4400 180) (effects (font (size 0.95 0.95)) (justify right)) (property "Intersheetrefs" "${INTERSHEET_REFS}" (at 215.9000 218.4400 0) (hide yes) (effects (font (size 1.0 1.0)) )))
+(global_label "USB_CC3V3" (shape bidirectional) (at 215.9000 218.4400 180) (effects (font (size 0.95 0.95)) (justify right)) (property "Intersheetrefs" "${INTERSHEET_REFS}" (at 215.9000 218.4400 0) (hide yes) (effects (font (size 1.0 1.0)) )))
 (wire (pts (xy 243.8400 218.4400) (xy 251.4600 218.4400)) (stroke (width 0) (type default)))
 (global_label "USB_DEFAULT_N" (shape bidirectional) (at 251.4600 218.4400 0) (effects (font (size 0.95 0.95)) (justify left)) (property "Intersheetrefs" "${INTERSHEET_REFS}" (at 251.4600 218.4400 0) (hide yes) (effects (font (size 1.0 1.0)) )))
 (symbol (lib_id "CANView:CANView_communicator_C15") (at 325.1200 218.4400 0) (unit 1) (in_bom yes) (on_board yes) (dnp no) (property "Reference" "C15" (at 325.1200 210.8200 0)  (effects (font (size 1.0 1.0)) ))(property "Value" "100n" (at 325.1200 213.3600 0)  (effects (font (size 1.0 1.0)) ))(property "Footprint" "CANView:Capacitor_SMD__C_0402_1005Metric" (at 325.1200 218.4400 0) (hide yes) (effects (font (size 1.0 1.0)) ))(property "MPN" "GEN-C-0402-100n-16V-X7R" (at 325.1200 218.4400 0) (hide yes) (effects (font (size 1.0 1.0)) ))(property "Specification" "16V; ±10%; X7R; -55..125C; verify effective capacitance under DC bias" (at 325.1200 218.4400 0) (hide yes) (effects (font (size 1.0 1.0)) ))(property "Source" "" (at 325.1200 218.4400 0) (hide yes) (effects (font (size 1.0 1.0)) ))(property "Assembly" "FIT" (at 325.1200 218.4400 0) (hide yes) (effects (font (size 1.0 1.0)) ))(instances (project "communicator" (path "/c8ff26d1-0b80-520e-ae3f-45aa29bfe092/7c624ae8-5f0b-5909-af7f-eefe17ebe63c" (reference "C15") (unit 1)))))
 (wire (pts (xy 314.9600 218.4400) (xy 307.3400 218.4400)) (stroke (width 0) (type default)))
-(global_label "USB_VBUS" (shape bidirectional) (at 307.3400 218.4400 180) (effects (font (size 0.95 0.95)) (justify right)) (property "Intersheetrefs" "${INTERSHEET_REFS}" (at 307.3400 218.4400 0) (hide yes) (effects (font (size 1.0 1.0)) )))
+(global_label "USB_CC3V3" (shape bidirectional) (at 307.3400 218.4400 180) (effects (font (size 0.95 0.95)) (justify right)) (property "Intersheetrefs" "${INTERSHEET_REFS}" (at 307.3400 218.4400 0) (hide yes) (effects (font (size 1.0 1.0)) )))
 (wire (pts (xy 335.2800 218.4400) (xy 342.9000 218.4400)) (stroke (width 0) (type default)))
 (global_label "GND" (shape bidirectional) (at 342.9000 218.4400 0) (effects (font (size 0.95 0.95)) (justify left)) (property "Intersheetrefs" "${INTERSHEET_REFS}" (at 342.9000 218.4400 0) (hide yes) (effects (font (size 1.0 1.0)) )))
@@
 (global_label "USB_POWER_ALLOWED" (shape bidirectional) (at 287.0200 121.9200 0) (effects (font (size 0.95 0.95)) (justify left)) (property "Intersheetrefs" "${INTERSHEET_REFS}" (at 287.0200 121.9200 0) (hide yes) (effects (font (size 1.0 1.0)) )))
 (wire (pts (xy 279.4000 127.0000) (xy 287.0200 127.0000)) (stroke (width 0) (type default)))
-(global_label "USB_VBUS" (shape bidirectional) (at 287.0200 127.0000 0) (effects (font (size 0.95 0.95)) (justify left)) (property "Intersheetrefs" "${INTERSHEET_REFS}" (at 287.0200 127.0000 0) (hide yes) (effects (font (size 1.0 1.0)) )))
+(global_label "USB_CC3V3" (shape bidirectional) (at 287.0200 127.0000 0) (effects (font (size 0.95 0.95)) (justify left)) (property "Intersheetrefs" "${INTERSHEET_REFS}" (at 287.0200 127.0000 0) (hide yes) (effects (font (size 1.0 1.0)) )))
 (symbol (lib_id "CANView:CANView_communicator_C16") (at 50.8000 238.7600 0) (unit 1) (in_bom yes) (on_board yes) (dnp no) (property "Reference" "C16" (at 50.8000 231.1400 0)  (effects (font (size 1.0 1.0)) ))(property "Value" "100n" (at 50.8000 233.6800 0)  (effects (font (size 1.0 1.0)) ))(property "Footprint" "CANView:Capacitor_SMD__C_0402_1005Metric" (at 50.8000 238.7600 0) (hide yes) (effects (font (size 1.0 1.0)) ))(property "MPN" "GEN-C-0402-100n-16V-X7R" (at 50.8000 238.7600 0) (hide yes) (effects (font (size 1.0 1.0)) ))(property "Specification" "16V; ±10%; X7R; -55..125C; verify effective capacitance under DC bias" (at 50.8000 238.7600 0) (hide yes) (effects (font (size 1.0 1.0)) ))(property "Source" "" (at 50.8000 238.7600 0) (hide yes) (effects (font (size 1.0 1.0)) ))(property "Assembly" "FIT" (at 50.8000 238.7600 0) (hide yes) (effects (font (size 1.0 1.0)) ))(instances (project "communicator" (path "/c8ff26d1-0b80-520e-ae3f-45aa29bfe092/7c624ae8-5f0b-5909-af7f-eefe17ebe63c" (reference "C16") (unit 1)))))
 (wire (pts (xy 40.6400 238.7600) (xy 33.0200 238.7600)) (stroke (width 0) (type default)))
-(global_label "USB_VBUS" (shape bidirectional) (at 33.0200 238.7600 180) (effects (font (size 0.95 0.95)) (justify right)) (property "Intersheetrefs" "${INTERSHEET_REFS}" (at 33.0200 238.7600 0) (hide yes) (effects (font (size 1.0 1.0)) )))
+(global_label "USB_CC3V3" (shape bidirectional) (at 33.0200 238.7600 180) (effects (font (size 0.95 0.95)) (justify right)) (property "Intersheetrefs" "${INTERSHEET_REFS}" (at 33.0200 238.7600 0) (hide yes) (effects (font (size 1.0 1.0)) )))
 (wire (pts (xy 60.9600 238.7600) (xy 68.5800 238.7600)) (stroke (width 0) (type default)))
 (global_label "GND" (shape bidirectional) (at 68.5800 238.7600 0) (effects (font (size 0.95 0.95)) (justify left)) (property "Intersheetrefs" "${INTERSHEET_REFS}" (at 68.5800 238.7600 0) (hide yes) (effects (font (size 1.0 1.0)) )))
