File: hardware/communicator/kicad/01b_usb_limit.kicad_sch (KiCad schematic)
At the start: 5 parts, among them U3 TPS2553QDBVRQ1

Commit message: fix: close hardware rail-fault paths and sensor contract gaps
Parts:
- removed C17: 1u, CANView:Capacitor_SMD__C_0603_1608Metric, symbol CANView:CANView_communicator_C17
- removed C18: 1u, CANView:Capacitor_SMD__C_0603_1608Metric, symbol CANView:CANView_communicator_C18
- removed R13: 26.7k, CANView:Resistor_SMD__R_0402_1005Metric, symbol CANView:CANView_communicator_R13
- added C19: 1u, CANView:Capacitor_SMD__C_0603_1608Metric, symbol CANView:CANView_communicator_C19
- added C20: 1u, CANView:Capacitor_SMD__C_0603_1608Metric, symbol CANView:CANView_communicator_C20
- added R15: 10k, CANView:Resistor_SMD__R_0402_1005Metric, symbol CANView:CANView_communicator_R15
- R14: value 10k -> 26.7k; MPN GEN-R-0402-10k-1% -> GEN-R-0402-26.7k-1%
Connections:
- net GND: now also R14.2, C19.2, C20.2
- net USB_FAULT_N: now also R15.2; no longer R14.2
- net USB_ILIM: now also R14.1
- net USB_LIMITED: now also C20.1
- net USB_VBUS: now also C19.1, R15.1; no longer R14.1
Other:
- moved on the sheet: R14
