File: hardware/communicator/kicad/02_system_power.kicad_sch (KiCad schematic)
At the start: 12 parts, among them U4 TPS2116DRLR, U5 TPS629210DRLR

Commit message: fix: close hardware rail-fault paths and sensor contract gaps
Parts:
- removed C19: 1u, CANView:Capacitor_SMD__C_0603_1608Metric, symbol CANView:CANView_communicator_C19
- removed C20: 1u, CANView:Capacitor_SMD__C_0603_1608Metric, symbol CANView:CANView_communicator_C20
- removed R15: 100k, CANView:Resistor_SMD__R_0402_1005Metric, symbol CANView:CANView_communicator_R15
- added C23: 4.7u, CANView:Capacitor_SMD__C_0603_1608Metric, symbol CANView:CANView_communicator_C23
- added C24: 22u, CANView:Capacitor_SMD__C_0805_2012Metric, symbol CANView:CANView_communicator_C24
- added R20: 27.4k, CANView:Resistor_SMD__R_0402_1005Metric, symbol CANView:CANView_communicator_R20
- C21: value 4.7u -> 1u; MPN GEN-C-0603-4.7u-16V-X7R -> GEN-C-0603-1u-16V-X7R
- C22: value 22u -> 1u; footprint CANView:Capacitor_SMD__C_0805_2012Metric -> CANView:Capacitor_SMD__C_0603_1608Metric; MPN GEN-C-0805-22u-10V-X7R -> GEN-C-0603-1u-16V-X7R; Specification 10V; ±10%; X7R; -55..125C; verify effective capacitance und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 -> 16V; ±10%; X7R; -55..125C; verify effective capacitance und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
- R16: value 30.1k -> 100k; MPN GEN-R-0402-30.1k-1% -> GEN-R-0402-100k-1%
- R17: value 10k -> 30.1k; MPN GEN-R-0402-10k-1% -> GEN-R-0402-30.1k-1%
- R18: value 249k -> 10k; MPN GEN-R-0402-249k-1% -> GEN-R-0402-10k-1%
- R19: value 27.4k -> 249k; MPN GEN-R-0402-27.4k-1% -> GEN-R-0402-249k-1%
Connections:
- net 3V3: now also R18.1, C24.1; no longer C22.1, R17.1
- net AUTO5V: now also C21.1, R16.1
- net AUTO_PRIORITY: now also R16.2, R17.1; no longer R16.1
- net GND: now also R17.2, C23.2, C24.2, R20.2; no longer R16.2, R18.2
- net SYS5V: now also C23.1; no longer C21.1
- net SYS_MODE: now also R20.1; no longer R19.1
- net USB_LIMITED: now also C22.1
- net USB_SERVICE_SENSE: now also R18.2; no longer R17.2
- net VSET_3V3: now also R19.1; no longer R18.1
Other:
- moved on the sheet: C21, C22, R16, R17, R18, R19
