File: hardware/communicator/kicad/03_reset.kicad_sch (KiCad schematic)
At the start: 4 parts, among them SW1 RESET, U6 TLV803EA30DPWR

Commit message: fix: close hardware rail-fault paths and sensor contract gaps
Parts:
- removed C23: 100n, CANView:Capacitor_SMD__C_0402_1005Metric, symbol CANView:CANView_communicator_C23
- removed R20: 10k, CANView:Resistor_SMD__R_0402_1005Metric, symbol CANView:CANView_communicator_R20
- added C25: 100n, CANView:Capacitor_SMD__C_0402_1005Metric, symbol CANView:CANView_communicator_C25
- added R21: 10k, CANView:Resistor_SMD__R_0402_1005Metric, symbol CANView:CANView_communicator_R21
Connections:
- net 3V3: now also C25.1, R21.1
- net GND: now also C25.2
- net SYS_RESET_N: now also R21.2
Changed lines of the file:
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@@
 (wire (pts (xy 114.3000 55.8800) (xy 121.9200 55.8800)) (stroke (width 0) (type default)))
 (global_label "3V3" (shape bidirectional) (at 121.9200 55.8800 0) (effects (font (size 0.95 0.95)) (justify left)) (property "Intersheetrefs" "${INTERSHEET_REFS}" (at 121.9200 55.8800 0) (hide yes) (effects (font (size 1.0 1.0)) )))
-(symbol (lib_id "CANView:CANView_communicator_R20") (at 50.8000 96.5200 0) (unit 1) (in_bom yes) (on_board yes) (dnp no) (property "Reference" "R20" (at 50.8000 88.9000 0)  (effects (font (size 1.0 1.0)) ))(property "Value" "10k" (at 50.8000 91.4400 0)  (effects (font (size 1.0 1.0)) ))(property "Footprint" "CANView:Resistor_SMD__R_0402_1005Metric" (at 50.8000 96.5200 0) (hide yes) (effects (font (size 1.0 1.0)) ))(property "MPN" "GEN-R-0402-10k-1%" (at 50.8000 96.5200 0) (hide yes) (effects (font (size 1.0 1.0)) ))(property "Specification" "0.1W; 50V; ±1%; ±100ppm/K; -55..155C" (at 50.8000 96.5200 0) (hide yes) (effects (font (size 1.0 1.0)) ))(property "Source" "" (at 50.8000 96.5200 0) (hide yes) (effects (font (size 1.0 1.0)) ))(property "Assembly" "FIT" (at 50.8000 96.5200 0) (hide yes) (effects (font (size 1.0 1.0)) ))(instances (project "communicator" (path "/c8ff26d1-0b80-520e-ae3f-45aa29bfe092/b0c65eb6-8613-514f-ac78-8647e9d40bec" (reference "R20") (unit 1)))))
+(symbol (lib_id "CANView:CANView_communicator_R21") (at 50.8000 96.5200 0) (unit 1) (in_bom yes) (on_board yes) (dnp no) (property "Reference" "R21" (at 50.8000 88.9000 0)  (effects (font (size 1.0 1.0)) ))(property "Value" "10k" (at 50.8000 91.4400 0)  (effects (font (size 1.0 1.0)) ))(property "Footprint" "CANView:Resistor_SMD__R_0402_1005Metric" (at 50.8000 96.5200 0) (hide yes) (effects (font (size 1.0 1.0)) ))(property "MPN" "GEN-R-0402-10k-1%" (at 50.8000 96.5200 0) (hide yes) (effects (font (size 1.0 1.0)) ))(property "Specification" "0.1W; 50V; ±1%; ±100ppm/K; -55..155C" (at 50.8000 96.5200 0) (hide yes) (effects (font (size 1.0 1.0)) ))(property "Source" "" (at 50.8000 96.5200 0) (hide yes) (effects (font (size 1.0 1.0)) ))(property "Assembly" "FIT" (at 50.8000 96.5200 0) (hide yes) (effects (font (size 1.0 1.0)) ))(instances (project "communicator" (path "/c8ff26d1-0b80-520e-ae3f-45aa29bfe092/b0c65eb6-8613-514f-ac78-8647e9d40bec" (reference "R21") (unit 1)))))
 (wire (pts (xy 40.6400 96.5200) (xy 33.0200 96.5200)) (stroke (width 0) (type default)))
 (global_label "3V3" (shape bidirectional) (at 33.0200 96.5200 180) (effects (font (size 0.95 0.95)) (justify right)) (property "Intersheetrefs" "${INTERSHEET_REFS}" (at 33.0200 96.5200 0) (hide yes) (effects (font (size 1.0 1.0)) )))
 (wire (pts (xy 60.9600 96.5200) (xy 68.5800 96.5200)) (stroke (width 0) (type default)))
 (global_label "SYS_RESET_N" (shape bidirectional) (at 68.5800 96.5200 0) (effects (font (size 0.95 0.95)) (justify left)) (property "Intersheetrefs" "${INTERSHEET_REFS}" (at 68.5800 96.5200 0) (hide yes) (effects (font (size 1.0 1.0)) )))
-(symbol (lib_id "CANView:CANView_communicator_C23") (at 142.2400 96.5200 0) (unit 1) (in_bom yes) (on_board yes) (dnp no) (property "Reference" "C23" (at 142.2400 88.9000 0)  (effects (font (size 1.0 1.0)) ))(property "Value" "100n" (at 142.2400 91.4400 0)  (effects (font (size 1.0 1.0)) ))(property "Footprint" "CANView:Capacitor_SMD__C_0402_1005Metric" (at 142.2400 96.5200 0) (hide yes) (effects (font (size 1.0 1.0)) ))(property "MPN" "GEN-C-0402-100n-16V-X7R" (at 142.2400 96.5200 0) (hide yes) (effects (font (size 1.0 1.0)) ))(property "Specification" "16V; ±10%; X7R; -55..125C; verify effective capacitance under DC bias" (at 142.2400 96.5200 0) (hide yes) (effects (font (size 1.0 1.0)) ))(property "Source" "" (at 142.2400 96.5200 0) (hide yes) (effects (font (size 1.0 1.0)) ))(property "Assembly" "FIT" (at 142.2400 96.5200 0) (hide yes) (effects (font (size 1.0 1.0)) ))(instances (project "communicator" (path "/c8ff26d1-0b80-520e-ae3f-45aa29bfe092/b0c65eb6-8613-514f-ac78-8647e9d40bec" (reference "C23") (unit 1)))))
+(symbol (lib_id "CANView:CANView_communicator_C25") (at 142.2400 96.5200 0) (unit 1) (in_bom yes) (on_board yes) (dnp no) (property "Reference" "C25" (at 142.2400 88.9000 0)  (effects (font (size 1.0 1.0)) ))(property "Value" "100n" (at 142.2400 91.4400 0)  (effects (font (size 1.0 1.0)) ))(property "Footprint" "CANView:Capacitor_SMD__C_0402_1005Metric" (at 142.2400 96.5200 0) (hide yes) (effects (font (size 1.0 1.0)) ))(property "MPN" "GEN-C-0402-100n-16V-X7R" (at 142.2400 96.5200 0) (hide yes) (effects (font (size 1.0 1.0)) ))(property "Specification" "16V; ±10%; X7R; -55..125C; verify effective capacitance under DC bias" (at 142.2400 96.5200 0) (hide yes) (effects (font (size 1.0 1.0)) ))(property "Source" "" (at 142.2400 96.5200 0) (hide yes) (effects (font (size 1.0 1.0)) ))(property "Assembly" "FIT" (at 142.2400 96.5200 0) (hide yes) (effects (font (size 1.0 1.0)) ))(instances (project "communicator" (path "/c8ff26d1-0b80-520e-ae3f-45aa29bfe092/b0c65eb6-8613-514f-ac78-8647e9d40bec" (reference "C25") (unit 1)))))
 (wire (pts (xy 132.0800 96.5200) (xy 124.4600 96.5200)) (stroke (width 0) (type default)))
 (global_label "3V3" (shape bidirectional) (at 124.4600 96.5200 180) (effects (font (size 0.95 0.95)) (justify right)) (property "Intersheetrefs" "${INTERSHEET_REFS}" (at 124.4600 96.5200 0) (hide yes) (effects (font (size 1.0 1.0)) )))

Commit message: Design independent OTA recovery and update N16R8 hardware
Parts:
- SW1: Specification Momentary normally-open; shared MCU reset -> Momentary normally-open; Communicator drives both superviso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
Connections:
- net 3V3: no longer U6.2 (MR_N)
- net SYS_RESET_N renamed ESP_RESET_N
- net ESP_RESET_N: no longer SW1.1
- new net GLOBAL_RESET_N: SW1.1, U6.2 (MR_N)
Changed lines of the file:
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@@
 (symbol (lib_id "CANView:CANView_communicator_U6") (at 88.9000 55.8800 0) (unit 1) (in_bom yes) (on_board yes) (dnp no) (property "Reference" "U6" (at 88.9000 40.6400 0)  (effects (font (size 1.0 1.0)) ))(property "Value" "TLV803EA30DPWR" (at 88.9000 43.1800 0)  (effects (font (size 1.0 1.0)) ))(property "Footprint" "CANView:Package_SON__Texas_X2SON-5_0.8x0.8mm_P0.48mm" (at 88.9000 55.8800 0) (hide yes) (effects (font (size 1.0 1.0)) ))(property "MPN" "TLV803EA30DPWR" (at 88.9000 55.8800 0) (hide yes) (effects (font (size 1.0 1.0)) ))(property "Specification" "3.08V threshold;130..270ms release delay; active-low open-drain" (at 88.9000 55.8800 0) (hide yes) (effects (font (size 1.0 1.0)) ))(property "Source" "tlv803e:pp4-5,9; DPW pin3 PAD may be grounded" (at 88.9000 55.8800 0) (hide yes) (effects (font (size 1.0 1.0)) ))(property "Assembly" "FIT" (at 88.9000 55.8800 0) (hide yes) (effects (font (size 1.0 1.0)) ))(instances (project "communicator" (path "/c8ff26d1-0b80-520e-ae3f-45aa29bfe092/b0c65eb6-8613-514f-ac78-8647e9d40bec" (reference "U6") (unit 1)))))
 (wire (pts (xy 63.5000 50.8000) (xy 55.8800 50.8000)) (stroke (width 0) (type default)))
-(global_label "SYS_RESET_N" (shape bidirectional) (at 55.8800 50.8000 180) (effects (font (size 0.95 0.95)) (justify right)) (property "Intersheetrefs" "${INTERSHEET_REFS}" (at 55.8800 50.8000 0) (hide yes) (effects (font (size 1.0 1.0)) )))
+(global_label "ESP_RESET_N" (shape bidirectional) (at 55.8800 50.8000 180) (effects (font (size 0.95 0.95)) (justify right)) (property "Intersheetrefs" "${INTERSHEET_REFS}" (at 55.8800 50.8000 0) (hide yes) (effects (font (size 1.0 1.0)) )))
 (wire (pts (xy 63.5000 55.8800) (xy 55.8800 55.8800)) (stroke (width 0) (type default)))
-(global_label "3V3" (shape bidirectional) (at 55.8800 55.8800 180) (effects (font (size 0.95 0.95)) (justify right)) (property "Intersheetrefs" "${INTERSHEET_REFS}" (at 55.8800 55.8800 0) (hide yes) (effects (font (size 1.0 1.0)) )))
+(global_label "GLOBAL_RESET_N" (shape bidirectional) (at 55.8800 55.8800 180) (effects (font (size 0.95 0.95)) (justify right)) (property "Intersheetrefs" "${INTERSHEET_REFS}" (at 55.8800 55.8800 0) (hide yes) (effects (font (size 1.0 1.0)) )))
 (wire (pts (xy 63.5000 60.9600) (xy 55.8800 60.9600)) (stroke (width 0) (type default)))
 (global_label "GND" (shape bidirectional) (at 55.8800 60.9600 180) (effects (font (size 0.95 0.95)) (justify right)) (property "Intersheetrefs" "${INTERSHEET_REFS}" (at 55.8800 60.9600 0) (hide yes) (effects (font (size 1.0 1.0)) )))
@@
 (global_label "3V3" (shape bidirectional) (at 33.0200 96.5200 180) (effects (font (size 0.95 0.95)) (justify right)) (property "Intersheetrefs" "${INTERSHEET_REFS}" (at 33.0200 96.5200 0) (hide yes) (effects (font (size 1.0 1.0)) )))
 (wire (pts (xy 60.9600 96.5200) (xy 68.5800 96.5200)) (stroke (width 0) (type default)))
-(global_label "SYS_RESET_N" (shape bidirectional) (at 68.5800 96.5200 0) (effects (font (size 0.95 0.95)) (justify left)) (property "Intersheetrefs" "${INTERSHEET_REFS}" (at 68.5800 96.5200 0) (hide yes) (effects (font (size 1.0 1.0)) )))
+(global_label "ESP_RESET_N" (shape bidirectional) (at 68.5800 96.5200 0) (effects (font (size 0.95 0.95)) (justify left)) (property "Intersheetrefs" "${INTERSHEET_REFS}" (at 68.5800 96.5200 0) (hide yes) (effects (font (size 1.0 1.0)) )))
 (symbol (lib_id "CANView:CANView_communicator_C25") (at 142.2400 96.5200 0) (unit 1) (in_bom yes) (on_board yes) (dnp no) (property "Reference" "C25" (at 142.2400 88.9000 0)  (effects (font (size 1.0 1.0)) ))(property "Value" "100n" (at 142.2400 91.4400 0)  (effects (font (size 1.0 1.0)) ))(property "Footprint" "CANView:Capacitor_SMD__C_0402_1005Metric" (at 142.2400 96.5200 0) (hide yes) (effects (font (size 1.0 1.0)) ))(property "MPN" "GEN-C-0402-100n-16V-X7R" (at 142.2400 96.5200 0) (hide yes) (effects (font (size 1.0 1.0)) ))(property "Specification" "16V; ±10%; X7R; -55..125C; verify effective capacitance under DC bias" (at 142.2400 96.5200 0) (hide yes) (effects (font (size 1.0 1.0)) ))(property "Source" "" (at 142.2400 96.5200 0) (hide yes) (effects (font (size 1.0 1.0)) ))(property "Assembly" "FIT" (at 142.2400 96.5200 0) (hide yes) (effects (font (size 1.0 1.0)) ))(instances (project "communicator" (path "/c8ff26d1-0b80-520e-ae3f-45aa29bfe092/b0c65eb6-8613-514f-ac78-8647e9d40bec" (reference "C25") (unit 1)))))
 (wire (pts (xy 132.0800 96.5200) (xy 124.4600 96.5200)) (stroke (width 0) (type default)))
@@
 (wire (pts (xy 152.4000 96.5200) (xy 160.0200 96.5200)) (stroke (width 0) (type default)))
 (global_label "GND" (shape bidirectional) (at 160.0200 96.5200 0) (effects (font (size 0.95 0.95)) (justify left)) (property "Intersheetrefs" "${INTERSHEET_REFS}" (at 160.0200 96.5200 0) (hide yes) (effects (font (size 1.0 1.0)) )))
-(symbol (lib_id "CANView:CANView_communicator_SW1") (at 233.6800 96.5200 0) (unit 1) (in_bom yes) (on_board yes) (dnp no) (property "Reference" "SW1" (at 233.6800 88.9000 0)  (effects (font (size 1.0 1.0)) ))(property "Value" "RESET" (at 233.6800 91.4400 0)  (effects (font (size 1.0 1.0)) ))(property "Footprint" "CANView:Button_Switch_SMD__SW_SPST_TL3342" (at 233.6800 96.5200 0) (hide yes) (effects (font (size 1.0 1.0)) ))(property "MPN" "TL3342F160QG" (at 233.6800 96.5200 0) (hide yes) (effects (font (size 1.0 1.0)) ))(property "Specification" "Momentary normally-open; shared MCU reset" (at 233.6800 96.5200 0) (hide yes) (effects (font (size 1.0 1.0)) ))(property "Source" "" (at 233.6800 96.5200 0) (hide yes) (effects (font (size 1.0 1.0)) ))(property "Assembly" "FIT" (at 233.6800 96.5200 0) (hide yes) (effects (font (size 1.0 1.0)) ))(instances (project "communicator" (path "/c8ff26d1-0b80-520e-ae3f-45aa29bfe092/b0c65eb6-8613-514f-ac78-8647e9d40bec" (reference "SW1") (unit 1)))))
+(symbol (lib_id "CANView:CANView_communicator_SW1") (at 233.6800 96.5200 0) (unit 1) (in_bom yes) (on_board yes) (dnp no) (property "Reference" "SW1" (at 233.6800 88.9000 0)  (effects (font (size 1.0 1.0)) ))(property "Value" "RESET" (at 233.6800 91.4400 0)  (effects (font (size 1.0 1.0)) ))(property "Footprint" "CANView:Button_Switch_SMD__SW_SPST_TL3342" (at 233.6800 96.5200 0) (hide yes) (effects (font (size 1.0 1.0)) ))(property "MPN" "TL3342F160QG" (at 233.6800 96.5200 0) (hide yes) (effects (font (size 1.0 1.0)) ))(property "Specification" "Momentary normally-open; Communicator drives both supervisor MR inputs, never joins reset outputs" (at 233.6800 96.5200 0) (hide yes) (effects (font (size 1.0 1.0)) ))(property "Source" "" (at 233.6800 96.5200 0) (hide yes) (effects (font (size 1.0 1.0)) ))(property "Assembly" "FIT" (at 233.6800 96.5200 0) (hide yes) (effects (font (size 1.0 1.0)) ))(instances (project "communicator" (path "/c8ff26d1-0b80-520e-ae3f-45aa29bfe092/b0c65eb6-8613-514f-ac78-8647e9d40bec" (reference "SW1") (unit 1)))))
 (wire (pts (xy 223.5200 96.5200) (xy 215.9000 96.5200)) (stroke (width 0) (type default)))
-(global_label "SYS_RESET_N" (shape bidirectional) (at 215.9000 96.5200 180) (effects (font (size 0.95 0.95)) (justify right)) (property "Intersheetrefs" "${INTERSHEET_REFS}" (at 215.9000 96.5200 0) (hide yes) (effects (font (size 1.0 1.0)) )))
+(global_label "GLOBAL_RESET_N" (shape bidirectional) (at 215.9000 96.5200 180) (effects (font (size 0.95 0.95)) (justify right)) (property "Intersheetrefs" "${INTERSHEET_REFS}" (at 215.9000 96.5200 0) (hide yes) (effects (font (size 1.0 1.0)) )))
 (wire (pts (xy 243.8400 96.5200) (xy 251.4600 96.5200)) (stroke (width 0) (type default)))
 (global_label "GND" (shape bidirectional) (at 251.4600 96.5200 0) (effects (font (size 0.95 0.95)) (justify left)) (property "Intersheetrefs" "${INTERSHEET_REFS}" (at 251.4600 96.5200 0) (hide yes) (effects (font (size 1.0 1.0)) )))
