File: hardware/communicator/kicad/03b_phy_power.kicad_sch (KiCad schematic)
At the start: 7 parts, among them U12 TLV803EA30DPWR, U9 TPS7A2033PDBVR

Commit message: fix: close hardware rail-fault paths and sensor contract gaps
Parts:
- removed C24: 1u, CANView:Capacitor_SMD__C_0603_1608Metric, symbol CANView:CANView_communicator_C24
- removed C25: 2.2u, CANView:Capacitor_SMD__C_0603_1608Metric, symbol CANView:CANView_communicator_C25
- removed R21: 10k, CANView:Resistor_SMD__R_0402_1005Metric, symbol CANView:CANView_communicator_R21
- added C27: 2.2u, CANView:Capacitor_SMD__C_0603_1608Metric, symbol CANView:CANView_communicator_C27
- added C28: 100n, CANView:Capacitor_SMD__C_0402_1005Metric, symbol CANView:CANView_communicator_C28
- added R23: 4.7k, CANView:Resistor_SMD__R_0402_1005Metric, symbol CANView:CANView_communicator_R23
- C26: value 100n -> 1u; footprint CANView:Capacitor_SMD__C_0402_1005Metric -> CANView:Capacitor_SMD__C_0603_1608Metric; MPN GEN-C-0402-100n-16V-X7R -> GEN-C-0603-1u-16V-X7R
- R22: value 4.7k -> 10k; MPN GEN-R-0402-4.7k-1% -> GEN-R-0402-10k-1%
Connections:
- net AUTO5V: now also C26.1
- net GND: now also C27.2, C28.2, R23.2; no longer R22.2
- net PHY3V3: now also C27.1, C28.1, R23.1; no longer C26.1
- net PHY_RESET_N: now also R22.2
Other:
- moved on the sheet: C26, R22
