File: hardware/communicator/kicad/03c_auto_qualification.kicad_sch (KiCad schematic)
At the start: 13 parts, among them U13 TPS3700DDCR, U14 TPS389001DSER, U15 SN74LVC1G11DCKR

Commit message: fix: close hardware rail-fault paths and sensor contract gaps
Parts:
- removed C27: 100n, CANView:Capacitor_SMD__C_0402_1005Metric, symbol CANView:CANView_communicator_C27
- removed C28: 10n, CANView:Capacitor_SMD__C_0603_1608Metric, symbol CANView:CANView_communicator_C28
- removed R23: 190k, CANView:Resistor_SMD__R_0603_1608Metric, symbol CANView:CANView_communicator_R23
- added C31: 100n, CANView:Capacitor_SMD__C_0402_1005Metric, symbol CANView:CANView_communicator_C31
- added C32: 100n, CANView:Capacitor_SMD__C_0402_1005Metric, symbol CANView:CANView_communicator_C32
- added R29: 10k, CANView:Resistor_SMD__R_0402_1005Metric, symbol CANView:CANView_communicator_R29
- C30: value 100n -> 10n; footprint CANView:Capacitor_SMD__C_0402_1005Metric -> CANView:Capacitor_SMD__C_0603_1608Metric; MPN GEN-C-0402-100n-16V-X7R -> GEN-C-0603-10n-16V-C0G; Specification 16V; ±10%; X7R; -55..125C; verify effective capacitance und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 -> 16V; ±5%; C0G; -55..125C; verify effective capacitance unde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
- R24: value 10k -> 190k; footprint CANView:Resistor_SMD__R_0402_1005Metric -> CANView:Resistor_SMD__R_0603_1608Metric; MPN GEN-R-0402-10k-0.1% -> GEN-R-0603-190k-0.1%
- R25: MPN GEN-R-0402-10k-1% -> GEN-R-0402-10k-0.1%; Specification 0.1W; 50V; ±1%; ±100ppm/K; -55..155C -> 0.1W; 50V; ±0.1%; ±100ppm/K; -55..155C
- R26: value 32k -> 10k; footprint CANView:Resistor_SMD__R_0603_1608Metric -> CANView:Resistor_SMD__R_0402_1005Metric; MPN GEN-R-0603-32k-0.05% -> GEN-R-0402-10k-1%; Specification 0.1W; 50V; ±0.05%; ±10ppm/K; -55..155C -> 0.1W; 50V; ±1%; ±100ppm/K; -55..155C
- R27: value 10k -> 32k; MPN GEN-R-0603-10k-0.05% -> GEN-R-0603-32k-0.05%
- R28: footprint CANView:Resistor_SMD__R_0402_1005Metric -> CANView:Resistor_SMD__R_0603_1608Metric; MPN GEN-R-0402-10k-1% -> GEN-R-0603-10k-0.05%; Specification 0.1W; 50V; ±1%; ±100ppm/K; -55..155C -> 0.1W; 50V; ±0.05%; ±10ppm/K; -55..155C
Connections:
- net AUTO5V: now also R27.1; no longer R26.1
- net AUTO5_DELAY: now also C30.1
- net AUTO5_GOOD: now also R29.2; no longer R28.2
- net AUTO5_SENSE: now also R27.2, R28.1; no longer R26.2, R27.1
- net BATT_GOOD: now also R26.2; no longer R25.2
- net BATT_SENSE: now also R24.2, R25.1; no longer R24.1
- net GND: now also R25.2, R28.2, C31.2, C32.2; no longer R24.2, R27.2
- net PHY3V3: now also R26.1, C31.1, C32.1, R29.1; no longer C30.1, R25.1, R28.1
- net PROTECTED_VBAT: now also R24.1
Other:
- moved on the sheet: C29, C30, R24, R25, R26, R27, R28
