File: hardware/communicator/kicad/04_stm32.kicad_sch (KiCad schematic)
At the start: 18 parts, among them U10 STM32G474CEU6

Commit message: feat: add R1 detailed hardware and navigation protocol review candidate
Parts:
- removed C1: 100n, CANView:Capacitor_SMD__C_0402_1005Metric, symbol CANView:CANView_communicator_C1
- removed C2: 100n, CANView:Capacitor_SMD__C_0402_1005Metric, symbol CANView:CANView_communicator_C2
- removed C3: 100n, CANView:Capacitor_SMD__C_0402_1005Metric, symbol CANView:CANView_communicator_C3
- removed C4: 4.7u, CANView:Capacitor_SMD__C_0603_1608Metric, symbol CANView:CANView_communicator_C4
- removed C5: 100n, CANView:Capacitor_SMD__C_0402_1005Metric, symbol CANView:CANView_communicator_C5
- removed C6: 1u, CANView:Capacitor_SMD__C_0603_1608Metric, symbol CANView:CANView_communicator_C6
- removed C7: 100n, CANView:Capacitor_SMD__C_0402_1005Metric, symbol CANView:CANView_communicator_C7
- removed R1: 0, CANView:Resistor_SMD__R_0402_1005Metric, symbol CANView:CANView_communicator_R1
- removed R10: 10k, CANView:Resistor_SMD__R_0402_1005Metric, symbol CANView:CANView_communicator_R10
- removed R2: 10k, CANView:Resistor_SMD__R_0402_1005Metric, symbol CANView:CANView_communicator_R2
- removed R3: 10k, CANView:Resistor_SMD__R_0402_1005Metric, symbol CANView:CANView_communicator_R3
- removed R4: 10k, CANView:Resistor_SMD__R_0402_1005Metric, symbol CANView:CANView_communicator_R4
- removed R5: 10k, CANView:Resistor_SMD__R_0402_1005Metric, symbol CANView:CANView_communicator_R5
- removed R6: 10k, CANView:Resistor_SMD__R_0402_1005Metric, symbol CANView:CANView_communicator_R6
- removed R7: 10k, CANView:Resistor_SMD__R_0402_1005Metric, symbol CANView:CANView_communicator_R7
- removed R8: 10k, CANView:Resistor_SMD__R_0402_1005Metric, symbol CANView:CANView_communicator_R8
- removed R9: 10k, CANView:Resistor_SMD__R_0402_1005Metric, symbol CANView:CANView_communicator_R9
- added C34: 100n, CANView:Capacitor_SMD__C_0402_1005Metric, symbol CANView:CANView_communicator_C34
- added C35: 100n, CANView:Capacitor_SMD__C_0402_1005Metric, symbol CANView:CANView_communicator_C35
- added C36: 100n, CANView:Capacitor_SMD__C_0402_1005Metric, symbol CANView:CANView_communicator_C36
- added C37: 4.7u, CANView:Capacitor_SMD__C_0603_1608Metric, symbol CANView:CANView_communicator_C37
- added C38: 100n, CANView:Capacitor_SMD__C_0402_1005Metric, symbol CANView:CANView_communicator_C38
- added C39: 1u, CANView:Capacitor_SMD__C_0603_1608Metric, symbol CANView:CANView_communicator_C39
- added C40: 100n, CANView:Capacitor_SMD__C_0402_1005Metric, symbol CANView:CANView_communicator_C40
- added R33: 0, CANView:Resistor_SMD__R_0402_1005Metric, symbol CANView:CANView_communicator_R33
- added R34: 10k, CANView:Resistor_SMD__R_0402_1005Metric, symbol CANView:CANView_communicator_R34
- added R35: 10k, CANView:Resistor_SMD__R_0402_1005Metric, symbol CANView:CANView_communicator_R35
- added R36: 10k, CANView:Resistor_SMD__R_0402_1005Metric, symbol CANView:CANView_communicator_R36
- added R37: 10k, CANView:Resistor_SMD__R_0402_1005Metric, symbol CANView:CANView_communicator_R37
- added R38: 10k, CANView:Resistor_SMD__R_0402_1005Metric, symbol CANView:CANView_communicator_R38
- added R39: 10k, CANView:Resistor_SMD__R_0402_1005Metric, symbol CANView:CANView_communicator_R39
- added R40: 10k, CANView:Resistor_SMD__R_0402_1005Metric, symbol CANView:CANView_communicator_R40
- added R41: 10k, CANView:Resistor_SMD__R_0402_1005Metric, symbol CANView:CANView_communicator_R41
- added R42: 10k, CANView:Resistor_SMD__R_0402_1005Metric, symbol CANView:CANView_communicator_R42
- U10: Source stm32g474: UFQFPN48 pinout, AF9/AF11/AF7; stm32g4-hardware -> stm32g474: UFQFPN48 pinout, AF9/AF11/AF7; pin 7 PG10-NRST r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
Connections:
- net 3V3: now also C34.1, C35.1, C36.1, C37.1, C38.1, R33.1, R37.1, R38.1, R39.1, R40.1, R41.1
- net BOOT0: now also R34.1
- net CAN1_TX_REQ: now also R37.2
- net CAN2_TX_REQ: now also R38.2
- net CAN3_TX_REQ: now also R39.2
- net FT_EN_REQ: now also R42.1
- net GND: now also C34.2, C35.2, C36.2, C37.2, C38.2, C39.2, C40.2, R34.2, R35.2, R36.2, R42.2
- net STB1_REQ: now also R40.2
- net STB2_REQ: now also R41.2
- net STM_ARM_EDGE: now also R35.1
- net VDDA: now also C39.1, C40.1, R33.2
- net WD_PULSE: now also R36.1
Other:
- note added: "STM32G474CEU6 / UFQFPN48. Pin 7 is the PG10-NRST dual-function reset pad. HSE 16MHz. USART2 4Mbps RTS/CTS. SWD only; USB pins are CAN1."
- note removed: "STM32G474CEU6 / UFQFPN48. HSE 16MHz. USART2 4Mbps RTS/CTS. SWD only; USB pins are CAN1."

Commit message: fix: close hardware rail-fault paths and sensor contract gaps
Parts:
- removed C34: 100n, CANView:Capacitor_SMD__C_0402_1005Metric, symbol CANView:CANView_communicator_C34
- removed C35: 100n, CANView:Capacitor_SMD__C_0402_1005Metric, symbol CANView:CANView_communicator_C35
- removed R33: 0, CANView:Resistor_SMD__R_0402_1005Metric, symbol CANView:CANView_communicator_R33
- added C41: 1u, CANView:Capacitor_SMD__C_0603_1608Metric, symbol CANView:CANView_communicator_C41
- added C42: 100n, CANView:Capacitor_SMD__C_0402_1005Metric, symbol CANView:CANView_communicator_C42
- added R43: 10k, CANView:Resistor_SMD__R_0402_1005Metric, symbol CANView:CANView_communicator_R43
- C37: value 4.7u -> 100n; footprint CANView:Capacitor_SMD__C_0603_1608Metric -> CANView:Capacitor_SMD__C_0402_1005Metric; MPN GEN-C-0603-4.7u-16V-X7R -> GEN-C-0402-100n-16V-X7R
- C39: value 1u -> 4.7u; MPN GEN-C-0603-1u-16V-X7R -> GEN-C-0603-4.7u-16V-X7R
- R34: value 10k -> 0; MPN GEN-R-0402-10k-1% -> GEN-R-0402-0-1%
Connections:
- net 3V3: now also C39.1, C40.1, R34.1, R42.1; no longer R37.1
- net BOOT0: now also R35.1; no longer R34.1
- net CAN1_TX_REQ: now also R38.2; no longer R37.2
- net CAN2_TX_REQ: now also R39.2; no longer R38.2
- net CAN3_TX_REQ: now also R40.2; no longer R39.2
- net FT_EN_REQ: now also R43.1; no longer R42.1
- net GND: now also R37.2, C41.2, C42.2, R43.2; no longer R34.2, R42.2
- net STB1_REQ: now also R41.2; no longer R40.2
- net STB2_REQ: now also R42.2; no longer R41.2
- net STM_ARM_EDGE: now also R36.1; no longer R35.1
- net VDDA: now also R34.2, C41.1, C42.1; no longer C39.1, C40.1
- net WD_PULSE: now also R37.1; no longer R36.1
Other:
- moved on the sheet: C36, C37, C38, C39, C40, R34, R35, R36, R37, R38, R39, R40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

Commit message: Design independent OTA recovery and update N16R8 hardware
Connections:
- net STM_RECOVERY_N: now reaches U10.47 (PB9)
- net SYS_RESET_N renamed STM_RESET_N
- no-connect marks 18 -> 17
Changed lines of the file:
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@@
 (global_label "HSE_OUT" (shape bidirectional) (at 55.8800 76.2000 180) (effects (font (size 0.95 0.95)) (justify right)) (property "Intersheetrefs" "${INTERSHEET_REFS}" (at 55.8800 76.2000 0) (hide yes) (effects (font (size 1.0 1.0)) )))
 (wire (pts (xy 63.5000 81.2800) (xy 55.8800 81.2800)) (stroke (width 0) (type default)))
-(global_label "SYS_RESET_N" (shape bidirectional) (at 55.8800 81.2800 180) (effects (font (size 0.95 0.95)) (justify right)) (property "Intersheetrefs" "${INTERSHEET_REFS}" (at 55.8800 81.2800 0) (hide yes) (effects (font (size 1.0 1.0)) )))
+(global_label "STM_RESET_N" (shape bidirectional) (at 55.8800 81.2800 180) (effects (font (size 0.95 0.95)) (justify right)) (property "Intersheetrefs" "${INTERSHEET_REFS}" (at 55.8800 81.2800 0) (hide yes) (effects (font (size 1.0 1.0)) )))
 (wire (pts (xy 63.5000 86.3600) (xy 55.8800 86.3600)) (stroke (width 0) (type default)))
 (global_label "ESP_RTS" (shape bidirectional) (at 55.8800 86.3600 180) (effects (font (size 0.95 0.95)) (justify right)) (property "Intersheetrefs" "${INTERSHEET_REFS}" (at 55.8800 86.3600 0) (hide yes) (effects (font (size 1.0 1.0)) )))
@@
 (wire (pts (xy 114.3000 152.4000) (xy 121.9200 152.4000)) (stroke (width 0) (type default)))
 (global_label "BOOT0" (shape bidirectional) (at 121.9200 152.4000 0) (effects (font (size 0.95 0.95)) (justify left)) (property "Intersheetrefs" "${INTERSHEET_REFS}" (at 121.9200 152.4000 0) (hide yes) (effects (font (size 1.0 1.0)) )))
-(no_connect (at 114.3000 157.4800))
+(wire (pts (xy 114.3000 157.4800) (xy 121.9200 157.4800)) (stroke (width 0) (type default)))
+(global_label "STM_RECOVERY_N" (shape bidirectional) (at 121.9200 157.4800 0) (effects (font (size 0.95 0.95)) (justify left)) (property "Intersheetrefs" "${INTERSHEET_REFS}" (at 121.9200 157.4800 0) (hide yes) (effects (font (size 1.0 1.0)) )))
 (wire (pts (xy 114.3000 162.5600) (xy 121.9200 162.5600)) (stroke (width 0) (type default)))
 (global_label "3V3" (shape bidirectional) (at 121.9200 162.5600 0) (effects (font (size 0.95 0.95)) (justify left)) (property "Intersheetrefs" "${INTERSHEET_REFS}" (at 121.9200 162.5600 0) (hide yes) (effects (font (size 1.0 1.0)) )))
