File: hardware/communicator/kicad/12b_latch_clear.kicad_sch (KiCad schematic)
At the start: 4 parts, among them U32 SN74LVC1G74DCUR, U37 SN74LVC1G11DCKR

Commit message: fix: close hardware rail-fault paths and sensor contract gaps
Parts:
- removed C63: 100n, CANView:Capacitor_SMD__C_0402_1005Metric, symbol CANView:CANView_communicator_C63
- removed C64: 100n, CANView:Capacitor_SMD__C_0402_1005Metric, symbol CANView:CANView_communicator_C64
- added C65: 100n, CANView:Capacitor_SMD__C_0402_1005Metric, symbol CANView:CANView_communicator_C65
- added C66: 100n, CANView:Capacitor_SMD__C_0402_1005Metric, symbol CANView:CANView_communicator_C66
Connections:
- net GND: now also C65.2, C66.2
- net PHY3V3: now also C65.1, C66.1
Changed lines of the file:
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@@
 (wire (pts (xy 279.4000 60.9600) (xy 287.0200 60.9600)) (stroke (width 0) (type default)))
 (global_label "TX_ARM" (shape bidirectional) (at 287.0200 60.9600 0) (effects (font (size 0.95 0.95)) (justify left)) (property "Intersheetrefs" "${INTERSHEET_REFS}" (at 287.0200 60.9600 0) (hide yes) (effects (font (size 1.0 1.0)) )))
-(symbol (lib_id "CANView:CANView_communicator_C63") (at 50.8000 101.6000 0) (unit 1) (in_bom yes) (on_board yes) (dnp no) (property "Reference" "C63" (at 50.8000 93.9800 0)  (effects (font (size 1.0 1.0)) ))(property "Value" "100n" (at 50.8000 96.5200 0)  (effects (font (size 1.0 1.0)) ))(property "Footprint" "CANView:Capacitor_SMD__C_0402_1005Metric" (at 50.8000 101.6000 0) (hide yes) (effects (font (size 1.0 1.0)) ))(property "MPN" "GEN-C-0402-100n-16V-X7R" (at 50.8000 101.6000 0) (hide yes) (effects (font (size 1.0 1.0)) ))(property "Specification" "16V; ±10%; X7R; -55..125C; verify effective capacitance under DC bias" (at 50.8000 101.6000 0) (hide yes) (effects (font (size 1.0 1.0)) ))(property "Source" "" (at 50.8000 101.6000 0) (hide yes) (effects (font (size 1.0 1.0)) ))(property "Assembly" "FIT" (at 50.8000 101.6000 0) (hide yes) (effects (font (size 1.0 1.0)) ))(instances (project "communicator" (path "/c8ff26d1-0b80-520e-ae3f-45aa29bfe092/de6ce08b-810c-5dad-9219-b6ed2b65a363" (reference "C63") (unit 1)))))
+(symbol (lib_id "CANView:CANView_communicator_C65") (at 50.8000 101.6000 0) (unit 1) (in_bom yes) (on_board yes) (dnp no) (property "Reference" "C65" (at 50.8000 93.9800 0)  (effects (font (size 1.0 1.0)) ))(property "Value" "100n" (at 50.8000 96.5200 0)  (effects (font (size 1.0 1.0)) ))(property "Footprint" "CANView:Capacitor_SMD__C_0402_1005Metric" (at 50.8000 101.6000 0) (hide yes) (effects (font (size 1.0 1.0)) ))(property "MPN" "GEN-C-0402-100n-16V-X7R" (at 50.8000 101.6000 0) (hide yes) (effects (font (size 1.0 1.0)) ))(property "Specification" "16V; ±10%; X7R; -55..125C; verify effective capacitance under DC bias" (at 50.8000 101.6000 0) (hide yes) (effects (font (size 1.0 1.0)) ))(property "Source" "" (at 50.8000 101.6000 0) (hide yes) (effects (font (size 1.0 1.0)) ))(property "Assembly" "FIT" (at 50.8000 101.6000 0) (hide yes) (effects (font (size 1.0 1.0)) ))(instances (project "communicator" (path "/c8ff26d1-0b80-520e-ae3f-45aa29bfe092/de6ce08b-810c-5dad-9219-b6ed2b65a363" (reference "C65") (unit 1)))))
 (wire (pts (xy 40.6400 101.6000) (xy 33.0200 101.6000)) (stroke (width 0) (type default)))
 (global_label "PHY3V3" (shape bidirectional) (at 33.0200 101.6000 180) (effects (font (size 0.95 0.95)) (justify right)) (property "Intersheetrefs" "${INTERSHEET_REFS}" (at 33.0200 101.6000 0) (hide yes) (effects (font (size 1.0 1.0)) )))
@@
 (wire (pts (xy 114.3000 66.0400) (xy 121.9200 66.0400)) (stroke (width 0) (type default)))
 (global_label "PHY3V3" (shape bidirectional) (at 121.9200 66.0400 0) (effects (font (size 0.95 0.95)) (justify left)) (property "Intersheetrefs" "${INTERSHEET_REFS}" (at 121.9200 66.0400 0) (hide yes) (effects (font (size 1.0 1.0)) )))
-(symbol (lib_id "CANView:CANView_communicator_C64") (at 142.2400 101.6000 0) (unit 1) (in_bom yes) (on_board yes) (dnp no) (property "Reference" "C64" (at 142.2400 93.9800 0)  (effects (font (size 1.0 1.0)) ))(property "Value" "100n" (at 142.2400 96.5200 0)  (effects (font (size 1.0 1.0)) ))(property "Footprint" "CANView:Capacitor_SMD__C_0402_1005Metric" (at 142.2400 101.6000 0) (hide yes) (effects (font (size 1.0 1.0)) ))(property "MPN" "GEN-C-0402-100n-16V-X7R" (at 142.2400 101.6000 0) (hide yes) (effects (font (size 1.0 1.0)) ))(property "Specification" "16V; ±10%; X7R; -55..125C; verify effective capacitance under DC bias" (at 142.2400 101.6000 0) (hide yes) (effects (font (size 1.0 1.0)) ))(property "Source" "" (at 142.2400 101.6000 0) (hide yes) (effects (font (size 1.0 1.0)) ))(property "Assembly" "FIT" (at 142.2400 101.6000 0) (hide yes) (effects (font (size 1.0 1.0)) ))(instances (project "communicator" (path "/c8ff26d1-0b80-520e-ae3f-45aa29bfe092/de6ce08b-810c-5dad-9219-b6ed2b65a363" (reference "C64") (unit 1)))))
+(symbol (lib_id "CANView:CANView_communicator_C66") (at 142.2400 101.6000 0) (unit 1) (in_bom yes) (on_board yes) (dnp no) (property "Reference" "C66" (at 142.2400 93.9800 0)  (effects (font (size 1.0 1.0)) ))(property "Value" "100n" (at 142.2400 96.5200 0)  (effects (font (size 1.0 1.0)) ))(property "Footprint" "CANView:Capacitor_SMD__C_0402_1005Metric" (at 142.2400 101.6000 0) (hide yes) (effects (font (size 1.0 1.0)) ))(property "MPN" "GEN-C-0402-100n-16V-X7R" (at 142.2400 101.6000 0) (hide yes) (effects (font (size 1.0 1.0)) ))(property "Specification" "16V; ±10%; X7R; -55..125C; verify effective capacitance under DC bias" (at 142.2400 101.6000 0) (hide yes) (effects (font (size 1.0 1.0)) ))(property "Source" "" (at 142.2400 101.6000 0) (hide yes) (effects (font (size 1.0 1.0)) ))(property "Assembly" "FIT" (at 142.2400 101.6000 0) (hide yes) (effects (font (size 1.0 1.0)) ))(instances (project "communicator" (path "/c8ff26d1-0b80-520e-ae3f-45aa29bfe092/de6ce08b-810c-5dad-9219-b6ed2b65a363" (reference "C66") (unit 1)))))
 (wire (pts (xy 132.0800 101.6000) (xy 124.4600 101.6000)) (stroke (width 0) (type default)))
 (global_label "PHY3V3" (shape bidirectional) (at 124.4600 101.6000 180) (effects (font (size 0.95 0.95)) (justify right)) (property "Intersheetrefs" "${INTERSHEET_REFS}" (at 124.4600 101.6000 0) (hide yes) (effects (font (size 1.0 1.0)) )))
