File: hardware/communicator/kicad/14_can_connectors.kicad_sch (KiCad schematic)
At the start: 10 parts, among them J20 CAN BUS 1/2/3

Commit message: fix: close hardware rail-fault paths and sensor contract gaps
Parts:
- removed C68: 4.7n, CANView:Capacitor_SMD__C_0805_2012Metric, symbol CANView:CANView_communicator_C68
- removed C69: 4.7n, CANView:Capacitor_SMD__C_0805_2012Metric, symbol CANView:CANView_communicator_C69
- removed R70: 60.4, CANView:Resistor_SMD__R_0805_2012Metric, symbol CANView:CANView_communicator_R70
- removed R71: 60.4, CANView:Resistor_SMD__R_0805_2012Metric, symbol CANView:CANView_communicator_R71
- removed R72: 60.4, CANView:Resistor_SMD__R_0805_2012Metric, symbol CANView:CANView_communicator_R72
- added C70: 4.7n, CANView:Capacitor_SMD__C_0805_2012Metric, symbol CANView:CANView_communicator_C70
- added C71: 4.7n, CANView:Capacitor_SMD__C_0805_2012Metric, symbol CANView:CANView_communicator_C71
- added R74: 60.4, CANView:Resistor_SMD__R_0805_2012Metric, symbol CANView:CANView_communicator_R74
- added R75: 60.4, CANView:Resistor_SMD__R_0805_2012Metric, symbol CANView:CANView_communicator_R75
- added R76: 60.4, CANView:Resistor_SMD__R_0805_2012Metric, symbol CANView:CANView_communicator_R76
Connections:
- net CAN1_H: now also R73.1
- net CAN1_L: now also R74.1
- net CAN1_TERM: now also R73.2, C70.1, R74.2
- net CAN2_H: now also R75.1
- net CAN2_L: now also R76.1; no longer R73.1
- net CAN2_TERM: now also C71.1, R75.2, R76.2; no longer R73.2
- net GND: now also C70.2, C71.2
Other:
- moved on the sheet: R73
