File: hardware/communicator/kicad/15_gnss_ins.kicad_sch (KiCad schematic)
At the start: 6 parts, among them U40 MTI-7-5A-T

Commit message: fix: close hardware rail-fault paths and sensor contract gaps
Parts:
- removed C70: 470n, CANView:Capacitor_SMD__C_0402_1005Metric, symbol CANView:CANView_communicator_C70
- removed C71: 100n, CANView:Capacitor_SMD__C_0402_1005Metric, symbol CANView:CANView_communicator_C71
- removed R74: 10k, CANView:Resistor_SMD__R_0402_1005Metric, symbol CANView:CANView_communicator_R74
- added C73: 100n, CANView:Capacitor_SMD__C_0402_1005Metric, symbol CANView:CANView_communicator_C73
- added C74: 4.7u, CANView:Capacitor_SMD__C_0603_1608Metric, symbol CANView:CANView_communicator_C74
- added R77: 10k, CANView:Resistor_SMD__R_0402_1005Metric, symbol CANView:CANView_communicator_R77
- C72: value 4.7u -> 470n; footprint CANView:Capacitor_SMD__C_0603_1608Metric -> CANView:Capacitor_SMD__C_0402_1005Metric; MPN GEN-C-0603-4.7u-16V-X7R -> GEN-C-0402-470n-16V-X7R
Connections:
- net 3V3: now also C73.1, C74.1, R77.1; no longer C72.1
- net GND: now also C73.2, C74.2
- net IMU_CS_N: now also R77.2
- net IMU_VDDA: now also C72.1
Other:
- moved on the sheet: C72
