File: hardware/communicator/kicad/16_barometer.kicad_sch (KiCad schematic)
At the start: 4 parts, among them U41 BMP384

Commit message: fix: close hardware rail-fault paths and sensor contract gaps
Parts:
- removed C73: 100n, CANView:Capacitor_SMD__C_0402_1005Metric, symbol CANView:CANView_communicator_C73
- removed C74: 100n, CANView:Capacitor_SMD__C_0402_1005Metric, symbol CANView:CANView_communicator_C74
- removed R75: 10k, CANView:Resistor_SMD__R_0402_1005Metric, symbol CANView:CANView_communicator_R75
- added C75: 100n, CANView:Capacitor_SMD__C_0402_1005Metric, symbol CANView:CANView_communicator_C75
- added C76: 100n, CANView:Capacitor_SMD__C_0402_1005Metric, symbol CANView:CANView_communicator_C76
- added R78: 10k, CANView:Resistor_SMD__R_0402_1005Metric, symbol CANView:CANView_communicator_R78
Connections:
- net 3V3: now also C75.1, C76.1, R78.1
- net BARO_CS_N: now also R78.2
- net GND: now also C75.2, C76.2
Changed lines of the file:
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@@
 (wire (pts (xy 114.3000 71.1200) (xy 121.9200 71.1200)) (stroke (width 0) (type default)))
 (global_label "3V3" (shape bidirectional) (at 121.9200 71.1200 0) (effects (font (size 0.95 0.95)) (justify left)) (property "Intersheetrefs" "${INTERSHEET_REFS}" (at 121.9200 71.1200 0) (hide yes) (effects (font (size 1.0 1.0)) )))
-(symbol (lib_id "CANView:CANView_communicator_C73") (at 50.8000 106.6800 0) (unit 1) (in_bom yes) (on_board yes) (dnp no) (property "Reference" "C73" (at 50.8000 99.0600 0)  (effects (font (size 1.0 1.0)) ))(property "Value" "100n" (at 50.8000 101.6000 0)  (effects (font (size 1.0 1.0)) ))(property "Footprint" "CANView:Capacitor_SMD__C_0402_1005Metric" (at 50.8000 106.6800 0) (hide yes) (effects (font (size 1.0 1.0)) ))(property "MPN" "GEN-C-0402-100n-16V-X7R" (at 50.8000 106.6800 0) (hide yes) (effects (font (size 1.0 1.0)) ))(property "Specification" "16V; ±10%; X7R; -55..125C; verify effective capacitance under DC bias" (at 50.8000 106.6800 0) (hide yes) (effects (font (size 1.0 1.0)) ))(property "Source" "" (at 50.8000 106.6800 0) (hide yes) (effects (font (size 1.0 1.0)) ))(property "Assembly" "FIT" (at 50.8000 106.6800 0) (hide yes) (effects (font (size 1.0 1.0)) ))(instances (project "communicator" (path "/c8ff26d1-0b80-520e-ae3f-45aa29bfe092/ba4727b2-cb38-5c92-94fb-646f2fe923d6" (reference "C73") (unit 1)))))
+(symbol (lib_id "CANView:CANView_communicator_C75") (at 50.8000 106.6800 0) (unit 1) (in_bom yes) (on_board yes) (dnp no) (property "Reference" "C75" (at 50.8000 99.0600 0)  (effects (font (size 1.0 1.0)) ))(property "Value" "100n" (at 50.8000 101.6000 0)  (effects (font (size 1.0 1.0)) ))(property "Footprint" "CANView:Capacitor_SMD__C_0402_1005Metric" (at 50.8000 106.6800 0) (hide yes) (effects (font (size 1.0 1.0)) ))(property "MPN" "GEN-C-0402-100n-16V-X7R" (at 50.8000 106.6800 0) (hide yes) (effects (font (size 1.0 1.0)) ))(property "Specification" "16V; ±10%; X7R; -55..125C; verify effective capacitance under DC bias" (at 50.8000 106.6800 0) (hide yes) (effects (font (size 1.0 1.0)) ))(property "Source" "" (at 50.8000 106.6800 0) (hide yes) (effects (font (size 1.0 1.0)) ))(property "Assembly" "FIT" (at 50.8000 106.6800 0) (hide yes) (effects (font (size 1.0 1.0)) ))(instances (project "communicator" (path "/c8ff26d1-0b80-520e-ae3f-45aa29bfe092/ba4727b2-cb38-5c92-94fb-646f2fe923d6" (reference "C75") (unit 1)))))
 (wire (pts (xy 40.6400 106.6800) (xy 33.0200 106.6800)) (stroke (width 0) (type default)))
 (global_label "3V3" (shape bidirectional) (at 33.0200 106.6800 180) (effects (font (size 0.95 0.95)) (justify right)) (property "Intersheetrefs" "${INTERSHEET_REFS}" (at 33.0200 106.6800 0) (hide yes) (effects (font (size 1.0 1.0)) )))
 (wire (pts (xy 60.9600 106.6800) (xy 68.5800 106.6800)) (stroke (width 0) (type default)))
 (global_label "GND" (shape bidirectional) (at 68.5800 106.6800 0) (effects (font (size 0.95 0.95)) (justify left)) (property "Intersheetrefs" "${INTERSHEET_REFS}" (at 68.5800 106.6800 0) (hide yes) (effects (font (size 1.0 1.0)) )))
-(symbol (lib_id "CANView:CANView_communicator_C74") (at 142.2400 106.6800 0) (unit 1) (in_bom yes) (on_board yes) (dnp no) (property "Reference" "C74" (at 142.2400 99.0600 0)  (effects (font (size 1.0 1.0)) ))(property "Value" "100n" (at 142.2400 101.6000 0)  (effects (font (size 1.0 1.0)) ))(property "Footprint" "CANView:Capacitor_SMD__C_0402_1005Metric" (at 142.2400 106.6800 0) (hide yes) (effects (font (size 1.0 1.0)) ))(property "MPN" "GEN-C-0402-100n-16V-X7R" (at 142.2400 106.6800 0) (hide yes) (effects (font (size 1.0 1.0)) ))(property "Specification" "16V; ±10%; X7R; -55..125C; verify effective capacitance under DC bias" (at 142.2400 106.6800 0) (hide yes) (effects (font (size 1.0 1.0)) ))(property "Source" "" (at 142.2400 106.6800 0) (hide yes) (effects (font (size 1.0 1.0)) ))(property "Assembly" "FIT" (at 142.2400 106.6800 0) (hide yes) (effects (font (size 1.0 1.0)) ))(instances (project "communicator" (path "/c8ff26d1-0b80-520e-ae3f-45aa29bfe092/ba4727b2-cb38-5c92-94fb-646f2fe923d6" (reference "C74") (unit 1)))))
+(symbol (lib_id "CANView:CANView_communicator_C76") (at 142.2400 106.6800 0) (unit 1) (in_bom yes) (on_board yes) (dnp no) (property "Reference" "C76" (at 142.2400 99.0600 0)  (effects (font (size 1.0 1.0)) ))(property "Value" "100n" (at 142.2400 101.6000 0)  (effects (font (size 1.0 1.0)) ))(property "Footprint" "CANView:Capacitor_SMD__C_0402_1005Metric" (at 142.2400 106.6800 0) (hide yes) (effects (font (size 1.0 1.0)) ))(property "MPN" "GEN-C-0402-100n-16V-X7R" (at 142.2400 106.6800 0) (hide yes) (effects (font (size 1.0 1.0)) ))(property "Specification" "16V; ±10%; X7R; -55..125C; verify effective capacitance under DC bias" (at 142.2400 106.6800 0) (hide yes) (effects (font (size 1.0 1.0)) ))(property "Source" "" (at 142.2400 106.6800 0) (hide yes) (effects (font (size 1.0 1.0)) ))(property "Assembly" "FIT" (at 142.2400 106.6800 0) (hide yes) (effects (font (size 1.0 1.0)) ))(instances (project "communicator" (path "/c8ff26d1-0b80-520e-ae3f-45aa29bfe092/ba4727b2-cb38-5c92-94fb-646f2fe923d6" (reference "C76") (unit 1)))))
 (wire (pts (xy 132.0800 106.6800) (xy 124.4600 106.6800)) (stroke (width 0) (type default)))
 (global_label "3V3" (shape bidirectional) (at 124.4600 106.6800 180) (effects (font (size 0.95 0.95)) (justify right)) (property "Intersheetrefs" "${INTERSHEET_REFS}" (at 124.4600 106.6800 0) (hide yes) (effects (font (size 1.0 1.0)) )))
 (wire (pts (xy 152.4000 106.6800) (xy 160.0200 106.6800)) (stroke (width 0) (type default)))
 (global_label "GND" (shape bidirectional) (at 160.0200 106.6800 0) (effects (font (size 0.95 0.95)) (justify left)) (property "Intersheetrefs" "${INTERSHEET_REFS}" (at 160.0200 106.6800 0) (hide yes) (effects (font (size 1.0 1.0)) )))
-(symbol (lib_id "CANView:CANView_communicator_R75") (at 233.6800 106.6800 0) (unit 1) (in_bom yes) (on_board yes) (dnp no) (property "Reference" "R75" (at 233.6800 99.0600 0)  (effects (font (size 1.0 1.0)) ))(property "Value" "10k" (at 233.6800 101.6000 0)  (effects (font (size 1.0 1.0)) ))(property "Footprint" "CANView:Resistor_SMD__R_0402_1005Metric" (at 233.6800 106.6800 0) (hide yes) (effects (font (size 1.0 1.0)) ))(property "MPN" "GEN-R-0402-10k-1%" (at 233.6800 106.6800 0) (hide yes) (effects (font (size 1.0 1.0)) ))(property "Specification" "0.1W; 50V; ±1%; ±100ppm/K; -55..155C" (at 233.6800 106.6800 0) (hide yes) (effects (font (size 1.0 1.0)) ))(property "Source" "" (at 233.6800 106.6800 0) (hide yes) (effects (font (size 1.0 1.0)) ))(property "Assembly" "FIT" (at 233.6800 106.6800 0) (hide yes) (effects (font (size 1.0 1.0)) ))(instances (project "communicator" (path "/c8ff26d1-0b80-520e-ae3f-45aa29bfe092/ba4727b2-cb38-5c92-94fb-646f2fe923d6" (reference "R75") (unit 1)))))
+(symbol (lib_id "CANView:CANView_communicator_R78") (at 233.6800 106.6800 0) (unit 1) (in_bom yes) (on_board yes) (dnp no) (property "Reference" "R78" (at 233.6800 99.0600 0)  (effects (font (size 1.0 1.0)) ))(property "Value" "10k" (at 233.6800 101.6000 0)  (effects (font (size 1.0 1.0)) ))(property "Footprint" "CANView:Resistor_SMD__R_0402_1005Metric" (at 233.6800 106.6800 0) (hide yes) (effects (font (size 1.0 1.0)) ))(property "MPN" "GEN-R-0402-10k-1%" (at 233.6800 106.6800 0) (hide yes) (effects (font (size 1.0 1.0)) ))(property "Specification" "0.1W; 50V; ±1%; ±100ppm/K; -55..155C" (at 233.6800 106.6800 0) (hide yes) (effects (font (size 1.0 1.0)) ))(property "Source" "" (at 233.6800 106.6800 0) (hide yes) (effects (font (size 1.0 1.0)) ))(property "Assembly" "FIT" (at 233.6800 106.6800 0) (hide yes) (effects (font (size 1.0 1.0)) ))(instances (project "communicator" (path "/c8ff26d1-0b80-520e-ae3f-45aa29bfe092/ba4727b2-cb38-5c92-94fb-646f2fe923d6" (reference "R78") (unit 1)))))
 (wire (pts (xy 223.5200 106.6800) (xy 215.9000 106.6800)) (stroke (width 0) (type default)))
 (global_label "3V3" (shape bidirectional) (at 215.9000 106.6800 180) (effects (font (size 0.95 0.95)) (justify right)) (property "Intersheetrefs" "${INTERSHEET_REFS}" (at 215.9000 106.6800 0) (hide yes) (effects (font (size 1.0 1.0)) )))
