File: hardware/communicator/kicad/17_gps_ports.kicad_sch (KiCad schematic)
At the start: 9 parts, among them J40 GNSS UART1 / GH10, J41 GNSS UART2 / PPS ONLY, U42 TPS7A2033PDBVR, U43 SN74LVC2G125DCUR

Commit message: fix: close hardware rail-fault paths and sensor contract gaps
Parts:
- removed C75: 1u, CANView:Capacitor_SMD__C_0603_1608Metric, symbol CANView:CANView_communicator_C75
- removed C76: 2.2u, CANView:Capacitor_SMD__C_0603_1608Metric, symbol CANView:CANView_communicator_C76
- removed R76: 33, CANView:Resistor_SMD__R_0402_1005Metric, symbol CANView:CANView_communicator_R76
- removed R77: 33, CANView:Resistor_SMD__R_0402_1005Metric, symbol CANView:CANView_communicator_R77
- added C78: 2.2u, CANView:Capacitor_SMD__C_0603_1608Metric, symbol CANView:CANView_communicator_C78
- added C79: 100n, CANView:Capacitor_SMD__C_0402_1005Metric, symbol CANView:CANView_communicator_C79
- added R79: 33, CANView:Resistor_SMD__R_0402_1005Metric, symbol CANView:CANView_communicator_R79
- added R80: 33, CANView:Resistor_SMD__R_0402_1005Metric, symbol CANView:CANView_communicator_R80
- C77: value 100n -> 1u; footprint CANView:Capacitor_SMD__C_0402_1005Metric -> CANView:Capacitor_SMD__C_0603_1608Metric; MPN GEN-C-0402-100n-16V-X7R -> GEN-C-0603-1u-16V-X7R
Connections:
- net GND: now also C78.2, C79.2
- net GPS3V3: now also C78.1, C79.1; no longer C77.1
- net GPS5V: now also C77.1
- net GPS_TX_SELECT: now also R80.1
- net GPS_TX_SELECTED: now also R79.2, R80.2
- net IMU_GPS_TX: now also R79.1
Other:
- moved on the sheet: C77
