File: hardware/communicator/kicad/18_gps_protection.kicad_sch (KiCad schematic)
At the start: 6 parts, among them U44 SN74LVC2G17DCKR

Commit message: fix: close hardware rail-fault paths and sensor contract gaps
Parts:
- removed C78: 100n, CANView:Capacitor_SMD__C_0402_1005Metric, symbol CANView:CANView_communicator_C78
- removed R78: 100k, CANView:Resistor_SMD__R_0402_1005Metric, symbol CANView:CANView_communicator_R78
- removed R79: 100k, CANView:Resistor_SMD__R_0402_1005Metric, symbol CANView:CANView_communicator_R79
- added C80: 100n, CANView:Capacitor_SMD__C_0402_1005Metric, symbol CANView:CANView_communicator_C80
- added R81: 100k, CANView:Resistor_SMD__R_0402_1005Metric, symbol CANView:CANView_communicator_R81
- added R82: 100k, CANView:Resistor_SMD__R_0402_1005Metric, symbol CANView:CANView_communicator_R82
Connections:
- net 3V3: now also C80.1
- net GND: now also C80.2, R81.2, R82.2
- net GPS_PPS_CONN: now also R82.1
- net GPS_TX_CONN: now also R81.1
Changed lines of the file:
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@@
 (wire (pts (xy 114.3000 60.9600) (xy 121.9200 60.9600)) (stroke (width 0) (type default)))
 (global_label "GPS_RX_TAP" (shape bidirectional) (at 121.9200 60.9600 0) (effects (font (size 0.95 0.95)) (justify left)) (property "Intersheetrefs" "${INTERSHEET_REFS}" (at 121.9200 60.9600 0) (hide yes) (effects (font (size 1.0 1.0)) )))
-(symbol (lib_id "CANView:CANView_communicator_C78") (at 50.8000 142.2400 0) (unit 1) (in_bom yes) (on_board yes) (dnp no) (property "Reference" "C78" (at 50.8000 134.6200 0)  (effects (font (size 1.0 1.0)) ))(property "Value" "100n" (at 50.8000 137.1600 0)  (effects (font (size 1.0 1.0)) ))(property "Footprint" "CANView:Capacitor_SMD__C_0402_1005Metric" (at 50.8000 142.2400 0) (hide yes) (effects (font (size 1.0 1.0)) ))(property "MPN" "GEN-C-0402-100n-16V-X7R" (at 50.8000 142.2400 0) (hide yes) (effects (font (size 1.0 1.0)) ))(property "Specification" "16V; ±10%; X7R; -55..125C; verify effective capacitance under DC bias" (at 50.8000 142.2400 0) (hide yes) (effects (font (size 1.0 1.0)) ))(property "Source" "" (at 50.8000 142.2400 0) (hide yes) (effects (font (size 1.0 1.0)) ))(property "Assembly" "FIT" (at 50.8000 142.2400 0) (hide yes) (effects (font (size 1.0 1.0)) ))(instances (project "communicator" (path "/c8ff26d1-0b80-520e-ae3f-45aa29bfe092/463ec372-39e9-56c1-a41f-ada528ed9f79" (reference "C78") (unit 1)))))
+(symbol (lib_id "CANView:CANView_communicator_C80") (at 50.8000 142.2400 0) (unit 1) (in_bom yes) (on_board yes) (dnp no) (property "Reference" "C80" (at 50.8000 134.6200 0)  (effects (font (size 1.0 1.0)) ))(property "Value" "100n" (at 50.8000 137.1600 0)  (effects (font (size 1.0 1.0)) ))(property "Footprint" "CANView:Capacitor_SMD__C_0402_1005Metric" (at 50.8000 142.2400 0) (hide yes) (effects (font (size 1.0 1.0)) ))(property "MPN" "GEN-C-0402-100n-16V-X7R" (at 50.8000 142.2400 0) (hide yes) (effects (font (size 1.0 1.0)) ))(property "Specification" "16V; ±10%; X7R; -55..125C; verify effective capacitance under DC bias" (at 50.8000 142.2400 0) (hide yes) (effects (font (size 1.0 1.0)) ))(property "Source" "" (at 50.8000 142.2400 0) (hide yes) (effects (font (size 1.0 1.0)) ))(property "Assembly" "FIT" (at 50.8000 142.2400 0) (hide yes) (effects (font (size 1.0 1.0)) ))(instances (project "communicator" (path "/c8ff26d1-0b80-520e-ae3f-45aa29bfe092/463ec372-39e9-56c1-a41f-ada528ed9f79" (reference "C80") (unit 1)))))
 (wire (pts (xy 40.6400 142.2400) (xy 33.0200 142.2400)) (stroke (width 0) (type default)))
 (global_label "3V3" (shape bidirectional) (at 33.0200 142.2400 180) (effects (font (size 0.95 0.95)) (justify right)) (property "Intersheetrefs" "${INTERSHEET_REFS}" (at 33.0200 142.2400 0) (hide yes) (effects (font (size 1.0 1.0)) )))
 (wire (pts (xy 60.9600 142.2400) (xy 68.5800 142.2400)) (stroke (width 0) (type default)))
 (global_label "GND" (shape bidirectional) (at 68.5800 142.2400 0) (effects (font (size 0.95 0.95)) (justify left)) (property "Intersheetrefs" "${INTERSHEET_REFS}" (at 68.5800 142.2400 0) (hide yes) (effects (font (size 1.0 1.0)) )))
-(symbol (lib_id "CANView:CANView_communicator_R78") (at 142.2400 142.2400 0) (unit 1) (in_bom yes) (on_board yes) (dnp no) (property "Reference" "R78" (at 142.2400 134.6200 0)  (effects (font (size 1.0 1.0)) ))(property "Value" "100k" (at 142.2400 137.1600 0)  (effects (font (size 1.0 1.0)) ))(property "Footprint" "CANView:Resistor_SMD__R_0402_1005Metric" (at 142.2400 142.2400 0) (hide yes) (effects (font (size 1.0 1.0)) ))(property "MPN" "GEN-R-0402-100k-1%" (at 142.2400 142.2400 0) (hide yes) (effects (font (size 1.0 1.0)) ))(property "Specification" "0.1W; 50V; ±1%; ±100ppm/K; -55..155C" (at 142.2400 142.2400 0) (hide yes) (effects (font (size 1.0 1.0)) ))(property "Source" "" (at 142.2400 142.2400 0) (hide yes) (effects (font (size 1.0 1.0)) ))(property "Assembly" "FIT" (at 142.2400 142.2400 0) (hide yes) (effects (font (size 1.0 1.0)) ))(instances (project "communicator" (path "/c8ff26d1-0b80-520e-ae3f-45aa29bfe092/463ec372-39e9-56c1-a41f-ada528ed9f79" (reference "R78") (unit 1)))))
+(symbol (lib_id "CANView:CANView_communicator_R81") (at 142.2400 142.2400 0) (unit 1) (in_bom yes) (on_board yes) (dnp no) (property "Reference" "R81" (at 142.2400 134.6200 0)  (effects (font (size 1.0 1.0)) ))(property "Value" "100k" (at 142.2400 137.1600 0)  (effects (font (size 1.0 1.0)) ))(property "Footprint" "CANView:Resistor_SMD__R_0402_1005Metric" (at 142.2400 142.2400 0) (hide yes) (effects (font (size 1.0 1.0)) ))(property "MPN" "GEN-R-0402-100k-1%" (at 142.2400 142.2400 0) (hide yes) (effects (font (size 1.0 1.0)) ))(property "Specification" "0.1W; 50V; ±1%; ±100ppm/K; -55..155C" (at 142.2400 142.2400 0) (hide yes) (effects (font (size 1.0 1.0)) ))(property "Source" "" (at 142.2400 142.2400 0) (hide yes) (effects (font (size 1.0 1.0)) ))(property "Assembly" "FIT" (at 142.2400 142.2400 0) (hide yes) (effects (font (size 1.0 1.0)) ))(instances (project "communicator" (path "/c8ff26d1-0b80-520e-ae3f-45aa29bfe092/463ec372-39e9-56c1-a41f-ada528ed9f79" (reference "R81") (unit 1)))))
 (wire (pts (xy 132.0800 142.2400) (xy 124.4600 142.2400)) (stroke (width 0) (type default)))
 (global_label "GPS_TX_CONN" (shape bidirectional) (at 124.4600 142.2400 180) (effects (font (size 0.95 0.95)) (justify right)) (property "Intersheetrefs" "${INTERSHEET_REFS}" (at 124.4600 142.2400 0) (hide yes) (effects (font (size 1.0 1.0)) )))
 (wire (pts (xy 152.4000 142.2400) (xy 160.0200 142.2400)) (stroke (width 0) (type default)))
 (global_label "GND" (shape bidirectional) (at 160.0200 142.2400 0) (effects (font (size 0.95 0.95)) (justify left)) (property "Intersheetrefs" "${INTERSHEET_REFS}" (at 160.0200 142.2400 0) (hide yes) (effects (font (size 1.0 1.0)) )))
-(symbol (lib_id "CANView:CANView_communicator_R79") (at 233.6800 142.2400 0) (unit 1) (in_bom yes) (on_board yes) (dnp no) (property "Reference" "R79" (at 233.6800 134.6200 0)  (effects (font (size 1.0 1.0)) ))(property "Value" "100k" (at 233.6800 137.1600 0)  (effects (font (size 1.0 1.0)) ))(property "Footprint" "CANView:Resistor_SMD__R_0402_1005Metric" (at 233.6800 142.2400 0) (hide yes) (effects (font (size 1.0 1.0)) ))(property "MPN" "GEN-R-0402-100k-1%" (at 233.6800 142.2400 0) (hide yes) (effects (font (size 1.0 1.0)) ))(property "Specification" "0.1W; 50V; ±1%; ±100ppm/K; -55..155C" (at 233.6800 142.2400 0) (hide yes) (effects (font (size 1.0 1.0)) ))(property "Source" "" (at 233.6800 142.2400 0) (hide yes) (effects (font (size 1.0 1.0)) ))(property "Assembly" "FIT" (at 233.6800 142.2400 0) (hide yes) (effects (font (size 1.0 1.0)) ))(instances (project "communicator" (path "/c8ff26d1-0b80-520e-ae3f-45aa29bfe092/463ec372-39e9-56c1-a41f-ada528ed9f79" (reference "R79") (unit 1)))))
+(symbol (lib_id "CANView:CANView_communicator_R82") (at 233.6800 142.2400 0) (unit 1) (in_bom yes) (on_board yes) (dnp no) (property "Reference" "R82" (at 233.6800 134.6200 0)  (effects (font (size 1.0 1.0)) ))(property "Value" "100k" (at 233.6800 137.1600 0)  (effects (font (size 1.0 1.0)) ))(property "Footprint" "CANView:Resistor_SMD__R_0402_1005Metric" (at 233.6800 142.2400 0) (hide yes) (effects (font (size 1.0 1.0)) ))(property "MPN" "GEN-R-0402-100k-1%" (at 233.6800 142.2400 0) (hide yes) (effects (font (size 1.0 1.0)) ))(property "Specification" "0.1W; 50V; ±1%; ±100ppm/K; -55..155C" (at 233.6800 142.2400 0) (hide yes) (effects (font (size 1.0 1.0)) ))(property "Source" "" (at 233.6800 142.2400 0) (hide yes) (effects (font (size 1.0 1.0)) ))(property "Assembly" "FIT" (at 233.6800 142.2400 0) (hide yes) (effects (font (size 1.0 1.0)) ))(instances (project "communicator" (path "/c8ff26d1-0b80-520e-ae3f-45aa29bfe092/463ec372-39e9-56c1-a41f-ada528ed9f79" (reference "R82") (unit 1)))))
 (wire (pts (xy 223.5200 142.2400) (xy 215.9000 142.2400)) (stroke (width 0) (type default)))
 (global_label "GPS_PPS_CONN" (shape bidirectional) (at 215.9000 142.2400 180) (effects (font (size 0.95 0.95)) (justify right)) (property "Intersheetrefs" "${INTERSHEET_REFS}" (at 215.9000 142.2400 0) (hide yes) (effects (font (size 1.0 1.0)) )))
