File: hardware/communicator/kicad/19_gps_power.kicad_sch (KiCad schematic)
At the start: 9 parts, among them U45 SN74LVC1G11DCKR, U46 TPS2553QDBVRQ1

Commit message: fix: close hardware rail-fault paths and sensor contract gaps
Parts:
- removed C31: 100n, CANView:Capacitor_SMD__C_0402_1005Metric, symbol CANView:CANView_communicator_C31
- removed C32: 1u, CANView:Capacitor_SMD__C_0603_1608Metric, symbol CANView:CANView_communicator_C32
- removed R29: 100k, CANView:Resistor_SMD__R_0402_1005Metric, symbol CANView:CANView_communicator_R29
- added C34: 1u, CANView:Capacitor_SMD__C_0603_1608Metric, symbol CANView:CANView_communicator_C34
- added C35: 1u, CANView:Capacitor_SMD__C_0603_1608Metric, symbol CANView:CANView_communicator_C35
- added R33: 4.7k, CANView:Resistor_SMD__R_0402_1005Metric, symbol CANView:CANView_communicator_R33
- C33: value 1u -> 100n; footprint CANView:Capacitor_SMD__C_0603_1608Metric -> CANView:Capacitor_SMD__C_0402_1005Metric; MPN GEN-C-0603-1u-16V-X7R -> GEN-C-0402-100n-16V-X7R
- R30: value 61.9k -> 100k; MPN GEN-R-0402-61.9k-1% -> GEN-R-0402-100k-1%
- R31: value 10k -> 61.9k; MPN GEN-R-0402-10k-1% -> GEN-R-0402-61.9k-1%
- R32: value 4.7k -> 10k; MPN GEN-R-0402-4.7k-1% -> GEN-R-0402-10k-1%
Connections:
- net AUTO5V: now also R32.1, C34.1; no longer R31.1
- net GND: now also R31.2, C34.2, C35.2, R33.2; no longer R32.2
- net GPS5V: now also C35.1, R33.1; no longer C33.1, R32.1
- net GPS_FAULT_N: now also R32.2; no longer R31.2
- net GPS_ILIM: now also R31.1; no longer R30.1
- net GPS_PWR_REQ: now also R30.1
- net PHY3V3: now also C33.1
Other:
- moved on the sheet: C33, R30, R31, R32

Commit message: Design independent OTA recovery and update N16R8 hardware
Connections:
- net SYS_RESET_N renamed RUN_ALLOWED
Changed lines of the file:
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@@
 (global_label "PHY3V3" (shape bidirectional) (at 121.9200 55.8800 0) (effects (font (size 0.95 0.95)) (justify left)) (property "Intersheetrefs" "${INTERSHEET_REFS}" (at 121.9200 55.8800 0) (hide yes) (effects (font (size 1.0 1.0)) )))
 (wire (pts (xy 114.3000 60.9600) (xy 121.9200 60.9600)) (stroke (width 0) (type default)))
-(global_label "SYS_RESET_N" (shape bidirectional) (at 121.9200 60.9600 0) (effects (font (size 0.95 0.95)) (justify left)) (property "Intersheetrefs" "${INTERSHEET_REFS}" (at 121.9200 60.9600 0) (hide yes) (effects (font (size 1.0 1.0)) )))
+(global_label "RUN_ALLOWED" (shape bidirectional) (at 121.9200 60.9600 0) (effects (font (size 0.95 0.95)) (justify left)) (property "Intersheetrefs" "${INTERSHEET_REFS}" (at 121.9200 60.9600 0) (hide yes) (effects (font (size 1.0 1.0)) )))
 (symbol (lib_id "CANView:CANView_communicator_C33") (at 50.8000 96.5200 0) (unit 1) (in_bom yes) (on_board yes) (dnp no) (property "Reference" "C33" (at 50.8000 88.9000 0)  (effects (font (size 1.0 1.0)) ))(property "Value" "100n" (at 50.8000 91.4400 0)  (effects (font (size 1.0 1.0)) ))(property "Footprint" "CANView:Capacitor_SMD__C_0402_1005Metric" (at 50.8000 96.5200 0) (hide yes) (effects (font (size 1.0 1.0)) ))(property "MPN" "GEN-C-0402-100n-16V-X7R" (at 50.8000 96.5200 0) (hide yes) (effects (font (size 1.0 1.0)) ))(property "Specification" "16V; ±10%; X7R; -55..125C; verify effective capacitance under DC bias" (at 50.8000 96.5200 0) (hide yes) (effects (font (size 1.0 1.0)) ))(property "Source" "" (at 50.8000 96.5200 0) (hide yes) (effects (font (size 1.0 1.0)) ))(property "Assembly" "FIT" (at 50.8000 96.5200 0) (hide yes) (effects (font (size 1.0 1.0)) ))(instances (project "communicator" (path "/c8ff26d1-0b80-520e-ae3f-45aa29bfe092/1f111898-addb-5e50-812f-b62538831c43" (reference "C33") (unit 1)))))
 (wire (pts (xy 40.6400 96.5200) (xy 33.0200 96.5200)) (stroke (width 0) (type default)))
