File: hardware/communicator/kicad/20_test_points.kicad_sch (KiCad schematic)
At the start: 24 parts

Commit message: Design independent OTA recovery and update N16R8 hardware
Parts:
- TP8: value SYS_RESET_N -> ESP_RESET_N
Connections:
- net SYS_RESET_N renamed ESP_RESET_N
Changed lines of the file:
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@@
 (wire (pts (xy 208.2800 60.9600) (xy 200.6600 60.9600)) (stroke (width 0) (type default)))
 (global_label "AUTO_GOOD" (shape bidirectional) (at 200.6600 60.9600 180) (effects (font (size 0.95 0.95)) (justify right)) (property "Intersheetrefs" "${INTERSHEET_REFS}" (at 200.6600 60.9600 0) (hide yes) (effects (font (size 1.0 1.0)) )))
-(symbol (lib_id "CANView:CANView_communicator_TP8") (at 325.1200 60.9600 0) (unit 1) (in_bom yes) (on_board yes) (dnp no) (property "Reference" "TP8" (at 325.1200 50.8000 0)  (effects (font (size 1.0 1.0)) ))(property "Value" "SYS_RESET_N" (at 325.1200 53.3400 0)  (effects (font (size 1.0 1.0)) ))(property "Footprint" "CANView:TestPoint__TestPoint_Pad_D1.0mm" (at 325.1200 60.9600 0) (hide yes) (effects (font (size 1.0 1.0)) ))(property "MPN" "PCB-PAD-1MM" (at 325.1200 60.9600 0) (hide yes) (effects (font (size 1.0 1.0)) ))(property "Specification" "Bare1mm probe pad; no purchased component; accessible with insulated probe" (at 325.1200 60.9600 0) (hide yes) (effects (font (size 1.0 1.0)) ))(property "Source" "PCB fabrication feature" (at 325.1200 60.9600 0) (hide yes) (effects (font (size 1.0 1.0)) ))(property "Assembly" "FIT" (at 325.1200 60.9600 0) (hide yes) (effects (font (size 1.0 1.0)) ))(instances (project "communicator" (path "/c8ff26d1-0b80-520e-ae3f-45aa29bfe092/4f63211f-ed62-58cf-b954-befba3d75c4e" (reference "TP8") (unit 1)))))
+(symbol (lib_id "CANView:CANView_communicator_TP8") (at 325.1200 60.9600 0) (unit 1) (in_bom yes) (on_board yes) (dnp no) (property "Reference" "TP8" (at 325.1200 50.8000 0)  (effects (font (size 1.0 1.0)) ))(property "Value" "ESP_RESET_N" (at 325.1200 53.3400 0)  (effects (font (size 1.0 1.0)) ))(property "Footprint" "CANView:TestPoint__TestPoint_Pad_D1.0mm" (at 325.1200 60.9600 0) (hide yes) (effects (font (size 1.0 1.0)) ))(property "MPN" "PCB-PAD-1MM" (at 325.1200 60.9600 0) (hide yes) (effects (font (size 1.0 1.0)) ))(property "Specification" "Bare1mm probe pad; no purchased component; accessible with insulated probe" (at 325.1200 60.9600 0) (hide yes) (effects (font (size 1.0 1.0)) ))(property "Source" "PCB fabrication feature" (at 325.1200 60.9600 0) (hide yes) (effects (font (size 1.0 1.0)) ))(property "Assembly" "FIT" (at 325.1200 60.9600 0) (hide yes) (effects (font (size 1.0 1.0)) ))(instances (project "communicator" (path "/c8ff26d1-0b80-520e-ae3f-45aa29bfe092/4f63211f-ed62-58cf-b954-befba3d75c4e" (reference "TP8") (unit 1)))))
 (wire (pts (xy 299.7200 60.9600) (xy 292.1000 60.9600)) (stroke (width 0) (type default)))
-(global_label "SYS_RESET_N" (shape bidirectional) (at 292.1000 60.9600 180) (effects (font (size 0.95 0.95)) (justify right)) (property "Intersheetrefs" "${INTERSHEET_REFS}" (at 292.1000 60.9600 0) (hide yes) (effects (font (size 1.0 1.0)) )))
+(global_label "ESP_RESET_N" (shape bidirectional) (at 292.1000 60.9600 180) (effects (font (size 0.95 0.95)) (justify right)) (property "Intersheetrefs" "${INTERSHEET_REFS}" (at 292.1000 60.9600 0) (hide yes) (effects (font (size 1.0 1.0)) )))
 (symbol (lib_id "CANView:CANView_communicator_TP9") (at 50.8000 81.2800 0) (unit 1) (in_bom yes) (on_board yes) (dnp no) (property "Reference" "TP9" (at 50.8000 71.1200 0)  (effects (font (size 1.0 1.0)) ))(property "Value" "PHY_RESET_N" (at 50.8000 73.6600 0)  (effects (font (size 1.0 1.0)) ))(property "Footprint" "CANView:TestPoint__TestPoint_Pad_D1.0mm" (at 50.8000 81.2800 0) (hide yes) (effects (font (size 1.0 1.0)) ))(property "MPN" "PCB-PAD-1MM" (at 50.8000 81.2800 0) (hide yes) (effects (font (size 1.0 1.0)) ))(property "Specification" "Bare1mm probe pad; no purchased component; accessible with insulated probe" (at 50.8000 81.2800 0) (hide yes) (effects (font (size 1.0 1.0)) ))(property "Source" "PCB fabrication feature" (at 50.8000 81.2800 0) (hide yes) (effects (font (size 1.0 1.0)) ))(property "Assembly" "FIT" (at 50.8000 81.2800 0) (hide yes) (effects (font (size 1.0 1.0)) ))(instances (project "communicator" (path "/c8ff26d1-0b80-520e-ae3f-45aa29bfe092/4f63211f-ed62-58cf-b954-befba3d75c4e" (reference "TP9") (unit 1)))))
 (wire (pts (xy 25.4000 81.2800) (xy 17.7800 81.2800)) (stroke (width 0) (type default)))
