File: hardware/communicator/kicad/23_ota_recovery.kicad_sch (KiCad schematic)
At the start: 9 parts, among them J32 ROM_BOOT authorization / OPEN, SW3 RECOVERY, U54 SN74LVC1G04DBVR, U55 SN74LVC1G11DCKR

Commit message: Fix OTA service interlock and durable activation policy
Parts:
- removed C85: 100n, CANView:Capacitor_SMD__C_0402_1005Metric, symbol CANView:CANView_communicator_C85
- removed R90: 10k, CANView:Resistor_SMD__R_0402_1005Metric, symbol CANView:CANView_communicator_R90
- removed R91: 10k, CANView:Resistor_SMD__R_0402_1005Metric, symbol CANView:CANView_communicator_R91
- added C87: 100n, CANView:Capacitor_SMD__C_0402_1005Metric, symbol CANView:CANView_communicator_C87
- added R93: 10k, CANView:Resistor_SMD__R_0402_1005Metric, symbol CANView:CANView_communicator_R93
- added R94: 1k, CANView:Resistor_SMD__R_0402_1005Metric, symbol CANView:CANView_communicator_R94
- R92: value 1k -> 10k; MPN GEN-R-0402-1k-1% -> GEN-R-0402-10k-1%
Connections:
- net 3V3: now also R92.1, C87.1
- net GND: now also C87.2, R93.2
- net RECOVERY_BUTTON_N: now also R92.2
- net ROM_BOOT_ALLOWED: now also R94.1; no longer R92.1
- net ROM_BOOT_LINK: now also R94.2; no longer R92.2
- net STM_BOOT0_REQ: now also R93.1
Other:
- moved on the sheet: C86, R92
