File: hardware/controller-adapter/kicad/01_waveshare_header.kicad_sch (KiCad schematic)
At the start: 3 parts, among them J1 Waveshare 2x16 mating male

Commit message: Design independent OTA recovery and update N16R8 hardware
Connections:
- net RECOVERY_BUTTON_N: now reaches J1.13 (GPIO41)
- net HOST_RESET_N: now reaches J1.22 (RESET)
- no-connect marks 22 -> 20
Changed lines of the file:
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@@
 (global_label "MIC_SD" (shape bidirectional) (at 55.8800 101.6000 180) (effects (font (size 0.95 0.95)) (justify right)) (property "Intersheetrefs" "${INTERSHEET_REFS}" (at 55.8800 101.6000 0) (hide yes) (effects (font (size 1.0 1.0)) )))
 (no_connect (at 63.5000 106.6800))
-(no_connect (at 63.5000 111.7600))
+(wire (pts (xy 63.5000 111.7600) (xy 55.8800 111.7600)) (stroke (width 0) (type default)))
+(global_label "RECOVERY_BUTTON_N" (shape bidirectional) (at 55.8800 111.7600 180) (effects (font (size 0.95 0.95)) (justify right)) (property "Intersheetrefs" "${INTERSHEET_REFS}" (at 55.8800 111.7600 0) (hide yes) (effects (font (size 1.0 1.0)) )))
 (no_connect (at 63.5000 116.8400))
 (no_connect (at 63.5000 121.9200))
@@
 (no_connect (at 114.3000 66.0400))
 (no_connect (at 114.3000 71.1200))
-(no_connect (at 114.3000 76.2000))
+(wire (pts (xy 114.3000 76.2000) (xy 121.9200 76.2000)) (stroke (width 0) (type default)))
+(global_label "HOST_RESET_N" (shape bidirectional) (at 121.9200 76.2000 0) (effects (font (size 0.95 0.95)) (justify left)) (property "Intersheetrefs" "${INTERSHEET_REFS}" (at 121.9200 76.2000 0) (hide yes) (effects (font (size 1.0 1.0)) )))
 (no_connect (at 114.3000 81.2800))
 (no_connect (at 114.3000 86.3600))
